File: PCB/PicoKeyboard/PicoKeyboard.kicad_pcb (KiCad board)
At the start: 2 copper layers, 361.9 x 133.3 mm, 171 parts, among them U1 Raspberry_Pi_Pico

Commit message: Update PCB
Parts:
- S1: value Keyswitch -> Esc
- S10: value Keyswitch -> F9
- S11: value Keyswitch -> F10
- S12: value Keyswitch -> F11
- S13: value Keyswitch -> F12
- S14: value Keyswitch -> Print
- S15: value Keyswitch -> Ins
- S16: value Keyswitch -> Del
- S17: value Keyswitch -> Tilde
- S18: value Keyswitch -> 1
- S19: value Keyswitch -> 2
- S2: value Keyswitch -> F1
- S20: value Keyswitch -> 3
- S21: value Keyswitch -> 4
- S22: value Keyswitch -> 5
- S23: value Keyswitch -> 6
- S24: value Keyswitch -> 7
- S25: value Keyswitch -> 8
- S26: value Keyswitch -> 9
- S27: value Keyswitch -> 0
- S28: value Keyswitch -> -; footprint Button_Switch_Keyboard:SW_Cherry_MX_2.00u_PCB -> Button_Switch_Keyboard:SW_Cherry_MX_1.00u_PCB
- S29: value Keyswitch -> =
- S3: value Keyswitch -> F2
- S30: value Keyswitch -> Backspace; footprint Button_Switch_Keyboard:SW_Cherry_MX_1.00u_PCB -> Button_Switch_Keyboard:SW_Cherry_MX_2.00u_PCB
- S31: value Keyswitch -> Home
- S32: value Keyswitch -> End; footprint Button_Switch_Keyboard:SW_Cherry_MX_1.50u_PCB -> Button_Switch_Keyboard:SW_Cherry_MX_1.00u_PCB
- S33: value Keyswitch -> Tab; footprint Button_Switch_Keyboard:SW_Cherry_MX_1.00u_PCB -> Button_Switch_Keyboard:SW_Cherry_MX_1.50u_PCB
- S34: value Keyswitch -> Q
- S35: value Keyswitch -> W
- S36: value Keyswitch -> E
- S37: value Keyswitch -> R
- S38: value Keyswitch -> T
- S39: value Keyswitch -> Y
- S4: value Keyswitch -> F3
- S40: value Keyswitch -> U
- S41: value Keyswitch -> I
- S42: value Keyswitch -> O
- S43: value Keyswitch -> P
- S44: value Keyswitch -> [
- S45: value Keyswitch -> ]; footprint Button_Switch_Keyboard:SW_Cherry_MX_1.50u_PCB -> Button_Switch_Keyboard:SW_Cherry_MX_1.00u_PCB
- S46: value Keyswitch -> \|; footprint Button_Switch_Keyboard:SW_Cherry_MX_1.00u_PCB -> Button_Switch_Keyboard:SW_Cherry_MX_1.50u_PCB
- S47: value Keyswitch -> PgDn
- S48: value Keyswitch -> CapsLock; footprint Button_Switch_Keyboard:SW_Cherry_MX_1.00u_PCB -> Button_Switch_Keyboard:SW_Cherry_MX_1.75u_PCB
- S49: value Keyswitch -> A; footprint Button_Switch_Keyboard:SW_Cherry_MX_1.75u_PCB -> Button_Switch_Keyboard:SW_Cherry_MX_1.00u_PCB
- S5: value Keyswitch -> F4
- S50: value Keyswitch -> S
- S51: value Keyswitch -> D
- S52: value Keyswitch -> F
- S53: value Keyswitch -> G
- S54: value Keyswitch -> H
- S55: value Keyswitch -> J
- S56: value Keyswitch -> K
- S57: value Keyswitch -> L
- S58: value Keyswitch -> ;:
- S59: value Keyswitch -> '"
- S6: value Keyswitch -> F5
- S60: value Keyswitch -> Enter; footprint Button_Switch_Keyboard:SW_Cherry_MX_1.00u_PCB -> Button_Switch_Keyboard:SW_Cherry_MX_2.25u_PCB
- S61: value Keyswitch -> PgUp; footprint Button_Switch_Keyboard:SW_Cherry_MX_2.25u_PCB -> Button_Switch_Keyboard:SW_Cherry_MX_1.00u_PCB
- S62: value Keyswitch -> L.Shift
- S63: value Keyswitch -> Z
- S64: value Keyswitch -> X
- S65: value Keyswitch -> C
- S66: value Keyswitch -> V
- S67: value Keyswitch -> B
- S68: value Keyswitch -> N
- S69: value Keyswitch -> M
- S7: value Keyswitch -> F6
- S70: value Keyswitch -> ,<
- S71: value Keyswitch -> .>
- S72: value Keyswitch -> /?
- S73: value Keyswitch -> R.Shift
- S74, S85: value Keyswitch -> Up
- S75: value Keyswitch -> L.Ctrl
- S76: value Keyswitch -> L.Super
- S77: value Keyswitch -> L.Alt
- S78: value Keyswitch -> Space
- S79: value Keyswitch -> Fn; footprint Button_Switch_Keyboard:SW_Cherry_MX_1.25u_PCB -> Button_Switch_Keyboard:SW_Cherry_MX_1.00u_PCB
- S8: value Keyswitch -> F7
- S80: value Keyswitch -> Custom 1; footprint Button_Switch_Keyboard:SW_Cherry_MX_1.25u_PCB -> Button_Switch_Keyboard:SW_Cherry_MX_1.00u_PCB
- S81: value Keyswitch -> Custom 2; footprint Button_Switch_Keyboard:SW_Cherry_MX_1.25u_PCB -> Button_Switch_Keyboard:SW_Cherry_MX_1.00u_PCB
- S82: value Keyswitch -> Custom 3; footprint Button_Switch_Keyboard:SW_Cherry_MX_1.25u_PCB -> Button_Switch_Keyboard:SW_Cherry_MX_1.00u_PCB
- S83: value Keyswitch -> Left
- S84: value Keyswitch -> Down
- S9: value Keyswitch -> F8
- moved D48 339.3 mm to (47.6, 126.2)
- moved S32 325.8 mm to (369.3, 75.9)
- moved S48 313.2 mm to (66.8, 114.0)
- moved S15 312.9 mm to (350.2, 52.1)
- moved S16 312.9 mm to (369.3, 52.1)
- moved D32 302.5 mm to (357.2, 88.1)
- moved D15 294.4 mm to (338.1, 64.3)
- moved D16 294.4 mm to (357.2, 64.3)
- moved D29 85.5 mm to (276.2, 88.1)
- moved D30 85.5 mm to (295.3, 88.1)
- moved D28 77.7 mm to (257.2, 88.1)
- moved D78 73.9 mm to (166.7, 164.3)
- moved S29 70.3 mm to (288.3, 75.9)
- moved S61 68.6 mm to (350.2, 114.0)
- moved D31 66.8 mm to (338.1, 88.1)
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Connections:
- D15 pad 1: R2 -> R1
- D16 pad 1: R2 -> R1
- D32 pad 1: R3 -> R2
- D48 pad 1: R3 -> R4
- S15 pad 1: C1 -> C15
- S16 pad 1: C2 -> C16
- S17 pad 1: C3 -> C1
- S18 pad 1: C4 -> C2
- S19 pad 1: C5 -> C3
- S20 pad 1: C6 -> C4
- S21 pad 1: C7 -> C5
- S22 pad 1: C8 -> C6
- S23 pad 1: C9 -> C7
- S24 pad 1: C10 -> C8
- S25 pad 1: C11 -> C9
- S26 pad 1: C12 -> C10
- S27 pad 1: C13 -> C11
- S28 pad 1: C14 -> C12
- S29 pad 1: C15 -> C13
- S30 pad 1: C16 -> C14
- S31 pad 1: C17 -> C15
- S32 pad 1: C1 -> C16
- S33 pad 1: C2 -> C1
- S34 pad 1: C3 -> C2
- S35 pad 1: C4 -> C3
- S36 pad 1: C5 -> C4
- S37 pad 1: C6 -> C5
- S38 pad 1: C7 -> C6
- S39 pad 1: C8 -> C7
- S40 pad 1: C9 -> C8
- S41 pad 1: C10 -> C9
- S42 pad 1: C11 -> C10
- S43 pad 1: C12 -> C11
- S44 pad 1: C13 -> C12
- S45 pad 1: C14 -> C13
- S46 pad 1: C15 -> C14
- S47 pad 1: C16 -> C15
- S48 pad 1: C17 -> C1
- S49 pad 1: C1 -> C2
- S50 pad 1: C2 -> C3
- S51 pad 1: C3 -> C4
- S52 pad 1: C4 -> C5
- S53 pad 1: C5 -> C6
- S54 pad 1: C6 -> C7
- S55 pad 1: C7 -> C8
- S56 pad 1: C8 -> C9
- S57 pad 1: C9 -> C10
- S58 pad 1: C10 -> C11
- S59 pad 1: C11 -> C12
- S60 pad 1: C12 -> C14
- S61 pad 1: C14 -> C15
- S74 pad 1: C16 -> C15
- S83 pad 1: C15 -> C14
- S84 pad 1: C16 -> C15
- S85 pad 1: C17 -> C16
Routing:
- net C1: track 444.4 -> 133.9 mm, vias 1 -> 0
- net C2: track 425.1 -> 137.8 mm, vias 1 -> 0
- net C3: track 397.1 -> 135.9 mm, vias 1 -> 0
- net C4: track 344.8 -> 107.1 mm, vias 1 -> 0
- net C5: track 352.3 -> 136.4 mm, vias 1 -> 0
- net C6: track 301.5 -> 104.7 mm, vias 1 -> 0
- net C8: track 321.6 -> 146.2 mm
- net C7: track 279.6 -> 104.7 mm, vias 1 -> 0
- net C9: track 301.4 -> 146.2 mm
- net C16: track 178.7 -> 23.8 mm
- net C17: track 142.4 -> 0.00 mm
- net C10: track 283.2 -> 147.5 mm
- net R6: track 453.5 -> 320.2 mm
- net C11: track 263.4 -> 146.1 mm
- net R4: track 400.2 -> 294.8 mm
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Other:
- board size 361.9 x 133.3 mm -> 352.4 x 133.4 mm

Commit message: New layout
Parts:
- removed D77, D78, D79, D80, D81, D82, D83, D84, D85: Diode, ScottoKeebs_Components:Diode_SOD-123
- removed S77: L.Alt, Button_Switch_Keyboard:SW_Cherry_MX_1.25u_PCB
- removed S78: Space, Button_Switch_Keyboard:SW_Cherry_MX_6.25u_PCB
- removed S79: Fn, Button_Switch_Keyboard:SW_Cherry_MX_1.00u_PCB
- removed S80: Custom 1, Button_Switch_Keyboard:SW_Cherry_MX_1.00u_PCB
- removed S81: Custom 2, Button_Switch_Keyboard:SW_Cherry_MX_1.00u_PCB
- removed S82: Custom 3, Button_Switch_Keyboard:SW_Cherry_MX_1.00u_PCB
- removed S83: Left, Button_Switch_Keyboard:SW_Cherry_MX_1.00u_PCB
- removed S84: Down, Button_Switch_Keyboard:SW_Cherry_MX_1.00u_PCB
- removed S85: Up, Button_Switch_Keyboard:SW_Cherry_MX_1.00u_PCB
- S1, S10, S11, S12, S13, S2, S3, S4, S5, S6, S7, S8, S9: footprint Button_Switch_Keyboard:SW_Cherry_MX_1.00u_PCB -> ScottoKeebs_MX:MX_PCB_1.00u
- S14: value Print -> Del; footprint Button_Switch_Keyboard:SW_Cherry_MX_1.00u_PCB -> ScottoKeebs_MX:MX_PCB_1.00u
- S15: value Ins -> Backtick; footprint Button_Switch_Keyboard:SW_Cherry_MX_1.00u_PCB -> ScottoKeebs_MX:MX_PCB_1.00u
- S16: value Del -> Num_1; footprint Button_Switch_Keyboard:SW_Cherry_MX_1.00u_PCB -> ScottoKeebs_MX:MX_PCB_1.00u
- S17: value Tilde -> Num_2; footprint Button_Switch_Keyboard:SW_Cherry_MX_1.00u_PCB -> ScottoKeebs_MX:MX_PCB_1.00u
- S18: value 1 -> Num_3; footprint Button_Switch_Keyboard:SW_Cherry_MX_1.00u_PCB -> ScottoKeebs_MX:MX_PCB_1.00u
- S19: value 2 -> Num_4; footprint Button_Switch_Keyboard:SW_Cherry_MX_1.00u_PCB -> ScottoKeebs_MX:MX_PCB_1.00u
- S20: value 3 -> Num_5; footprint Button_Switch_Keyboard:SW_Cherry_MX_1.00u_PCB -> ScottoKeebs_MX:MX_PCB_1.00u
- S21: value 4 -> Num_6; footprint Button_Switch_Keyboard:SW_Cherry_MX_1.00u_PCB -> ScottoKeebs_MX:MX_PCB_1.00u
- S22: value 5 -> Num_7; footprint Button_Switch_Keyboard:SW_Cherry_MX_1.00u_PCB -> ScottoKeebs_MX:MX_PCB_1.00u
- S23: value 6 -> Num_8; footprint Button_Switch_Keyboard:SW_Cherry_MX_1.00u_PCB -> ScottoKeebs_MX:MX_PCB_1.00u
- S24: value 7 -> Num_9; footprint Button_Switch_Keyboard:SW_Cherry_MX_1.00u_PCB -> ScottoKeebs_MX:MX_PCB_1.00u
- S25: value 8 -> Num_0; footprint Button_Switch_Keyboard:SW_Cherry_MX_1.00u_PCB -> ScottoKeebs_MX:MX_PCB_1.00u
- S26: value 9 -> Minus; footprint Button_Switch_Keyboard:SW_Cherry_MX_1.00u_PCB -> ScottoKeebs_MX:MX_PCB_1.00u
- S27: value 0 -> Add; footprint Button_Switch_Keyboard:SW_Cherry_MX_1.00u_PCB -> ScottoKeebs_MX:MX_PCB_1.00u
- S28: value - -> Backspace; footprint Button_Switch_Keyboard:SW_Cherry_MX_1.00u_PCB -> ScottoKeebs_MX:MX_PCB_2.00u
- S29: value = -> Tab; footprint Button_Switch_Keyboard:SW_Cherry_MX_1.00u_PCB -> ScottoKeebs_MX:MX_PCB_1.50u
- S30: value Backspace -> Q; footprint Button_Switch_Keyboard:SW_Cherry_MX_2.00u_PCB -> ScottoKeebs_MX:MX_PCB_1.00u
- S31: value Home -> W; footprint Button_Switch_Keyboard:SW_Cherry_MX_1.00u_PCB -> ScottoKeebs_MX:MX_PCB_1.00u
- S32: value End -> E; footprint Button_Switch_Keyboard:SW_Cherry_MX_1.00u_PCB -> ScottoKeebs_MX:MX_PCB_1.00u
- S33: value Tab -> R; footprint Button_Switch_Keyboard:SW_Cherry_MX_1.50u_PCB -> ScottoKeebs_MX:MX_PCB_1.00u
- S34: value Q -> T; footprint Button_Switch_Keyboard:SW_Cherry_MX_1.00u_PCB -> ScottoKeebs_MX:MX_PCB_1.00u
- S35: value W -> Y; footprint Button_Switch_Keyboard:SW_Cherry_MX_1.00u_PCB -> ScottoKeebs_MX:MX_PCB_1.00u
- S36: value E -> U; footprint Button_Switch_Keyboard:SW_Cherry_MX_1.00u_PCB -> ScottoKeebs_MX:MX_PCB_1.00u
- S37: value R -> I; footprint Button_Switch_Keyboard:SW_Cherry_MX_1.00u_PCB -> ScottoKeebs_MX:MX_PCB_1.00u
- S38: value T -> O; footprint Button_Switch_Keyboard:SW_Cherry_MX_1.00u_PCB -> ScottoKeebs_MX:MX_PCB_1.00u
- S39: value Y -> P; footprint Button_Switch_Keyboard:SW_Cherry_MX_1.00u_PCB -> ScottoKeebs_MX:MX_PCB_1.00u
- S40: value U -> [; footprint Button_Switch_Keyboard:SW_Cherry_MX_1.00u_PCB -> ScottoKeebs_MX:MX_PCB_1.00u
- S41: value I -> ]; footprint Button_Switch_Keyboard:SW_Cherry_MX_1.00u_PCB -> ScottoKeebs_MX:MX_PCB_1.00u
- S42: value O -> Pipe; footprint Button_Switch_Keyboard:SW_Cherry_MX_1.00u_PCB -> ScottoKeebs_MX:MX_PCB_1.50u
- S43: value P -> Caps; footprint Button_Switch_Keyboard:SW_Cherry_MX_1.00u_PCB -> ScottoKeebs_MX:MX_PCB_1.75u
- S44: value [ -> A; footprint Button_Switch_Keyboard:SW_Cherry_MX_1.00u_PCB -> ScottoKeebs_MX:MX_PCB_1.00u
- S45: value ] -> S; footprint Button_Switch_Keyboard:SW_Cherry_MX_1.00u_PCB -> ScottoKeebs_MX:MX_PCB_1.00u
- S46: value \| -> D; footprint Button_Switch_Keyboard:SW_Cherry_MX_1.50u_PCB -> ScottoKeebs_MX:MX_PCB_1.00u
- S47: value PgDn -> F; footprint Button_Switch_Keyboard:SW_Cherry_MX_1.00u_PCB -> ScottoKeebs_MX:MX_PCB_1.00u
- S48: value CapsLock -> G; footprint Button_Switch_Keyboard:SW_Cherry_MX_1.75u_PCB -> ScottoKeebs_MX:MX_PCB_1.00u
- S49: value A -> H; footprint Button_Switch_Keyboard:SW_Cherry_MX_1.00u_PCB -> ScottoKeebs_MX:MX_PCB_1.00u
- S50: value S -> J; footprint Button_Switch_Keyboard:SW_Cherry_MX_1.00u_PCB -> ScottoKeebs_MX:MX_PCB_1.00u
- S51: value D -> K; footprint Button_Switch_Keyboard:SW_Cherry_MX_1.00u_PCB -> ScottoKeebs_MX:MX_PCB_1.00u
- S52: value F -> L; footprint Button_Switch_Keyboard:SW_Cherry_MX_1.00u_PCB -> ScottoKeebs_MX:MX_PCB_1.00u
- S53: value G -> Semicolon; footprint Button_Switch_Keyboard:SW_Cherry_MX_1.00u_PCB -> ScottoKeebs_MX:MX_PCB_1.00u
- S54: value H -> Quote; footprint Button_Switch_Keyboard:SW_Cherry_MX_1.00u_PCB -> ScottoKeebs_MX:MX_PCB_1.00u
- S55: value J -> Enter; footprint Button_Switch_Keyboard:SW_Cherry_MX_1.00u_PCB -> ScottoKeebs_MX:MX_PCB_2.25u
- S56: value K -> L.Shift; footprint Button_Switch_Keyboard:SW_Cherry_MX_1.00u_PCB -> ScottoKeebs_MX:MX_PCB_2.25u
- S57: value L -> Z; footprint Button_Switch_Keyboard:SW_Cherry_MX_1.00u_PCB -> ScottoKeebs_MX:MX_PCB_1.00u
- S58: value ;: -> X; footprint Button_Switch_Keyboard:SW_Cherry_MX_1.00u_PCB -> ScottoKeebs_MX:MX_PCB_1.00u
- S59: value '" -> C; footprint Button_Switch_Keyboard:SW_Cherry_MX_1.00u_PCB -> ScottoKeebs_MX:MX_PCB_1.00u
- S60: value Enter -> V; footprint Button_Switch_Keyboard:SW_Cherry_MX_2.25u_PCB -> ScottoKeebs_MX:MX_PCB_1.00u
- S61: value PgUp -> B; footprint Button_Switch_Keyboard:SW_Cherry_MX_1.00u_PCB -> ScottoKeebs_MX:MX_PCB_1.00u
- S62: value L.Shift -> N; footprint Button_Switch_Keyboard:SW_Cherry_MX_2.25u_PCB -> ScottoKeebs_MX:MX_PCB_1.00u
- S63: value Z -> M; footprint Button_Switch_Keyboard:SW_Cherry_MX_1.00u_PCB -> ScottoKeebs_MX:MX_PCB_1.00u
- S64: value X -> Comma; footprint Button_Switch_Keyboard:SW_Cherry_MX_1.00u_PCB -> ScottoKeebs_MX:MX_PCB_1.00u
- S65: value C -> Period; footprint Button_Switch_Keyboard:SW_Cherry_MX_1.00u_PCB -> ScottoKeebs_MX:MX_PCB_1.00u
- S66: value V -> Slash; footprint Button_Switch_Keyboard:SW_Cherry_MX_1.00u_PCB -> ScottoKeebs_MX:MX_PCB_1.00u
- S67: value B -> R.Shift; footprint Button_Switch_Keyboard:SW_Cherry_MX_1.00u_PCB -> ScottoKeebs_MX:MX_PCB_2.75u
- S68: value N -> Ctrl; footprint Button_Switch_Keyboard:SW_Cherry_MX_1.00u_PCB -> ScottoKeebs_MX:MX_PCB_1.25u
- S69: value M -> Super; footprint Button_Switch_Keyboard:SW_Cherry_MX_1.00u_PCB -> ScottoKeebs_MX:MX_PCB_1.25u
- S70: value ,< -> Alt; footprint Button_Switch_Keyboard:SW_Cherry_MX_1.00u_PCB -> ScottoKeebs_MX:MX_PCB_1.25u
- S71: value .> -> Space; footprint Button_Switch_Keyboard:SW_Cherry_MX_1.00u_PCB -> ScottoKeebs_MX:MX_PCB_6.25u
- S72: value /? -> Fn; footprint Button_Switch_Keyboard:SW_Cherry_MX_1.00u_PCB -> ScottoKeebs_MX:MX_PCB_1.00u
- S73: value R.Shift -> Custom_1; footprint Button_Switch_Keyboard:SW_Cherry_MX_2.75u_PCB -> ScottoKeebs_MX:MX_PCB_1.00u
- S74: value Up -> Custom_2; footprint Button_Switch_Keyboard:SW_Cherry_MX_1.00u_PCB -> ScottoKeebs_MX:MX_PCB_1.00u
- S75: value L.Ctrl -> Custom_3; footprint Button_Switch_Keyboard:SW_Cherry_MX_1.25u_PCB -> ScottoKeebs_MX:MX_PCB_1.00u
- S76: value L.Super -> Custom_4; footprint Button_Switch_Keyboard:SW_Cherry_MX_1.25u_PCB -> ScottoKeebs_MX:MX_PCB_1.00u
- moved S15 283.7 mm to (71.4, 104.8)
- moved S16 283.7 mm to (90.5, 104.8)
- moved U1 275.3 mm to (111.7, 42.9), turned to 90 degrees
- moved S75 258.6 mm to (319.1, 181.0)
- moved S76 253.9 mm to (338.1, 181.0)
- moved S31 236.1 mm to (119.1, 123.8)
- moved S32 236.1 mm to (138.1, 123.8)
- moved S30 222.1 mm to (100.0, 123.8)
- moved D75 220.7 mm to (217.8, 23.8), turned to -90 degrees
- moved S29 217.4 mm to (76.2, 123.8)
- moved D76 208.1 mm to (225.0, 23.8), turned to -90 degrees
- moved D62 199.2 mm to (210.7, 30.9), turned to -90 degrees
- moved S47 194.3 mm to (161.9, 142.9)
- moved S43 187.4 mm to (78.6, 142.9)
- moved S46 185.1 mm to (142.9, 142.9)
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Connections:
- D1 pad 1: R1 -> R0
- D10 pad 1: R1 -> R0
- D11 pad 1: R1 -> R0
- D12 pad 1: R1 -> R0
- D13 pad 1: R1 -> R0
- D14 pad 1: R1 -> R3
- D17 pad 1: R2 -> R1
- D18 pad 1: R2 -> R1
- D19 pad 1: R2 -> R1
- D2 pad 1: R1 -> R0
- D20 pad 1: R2 -> R1
- D21 pad 1: R2 -> R1
- D22 pad 1: R2 -> R1
- D23 pad 1: R2 -> R1
- D24 pad 1: R2 -> R1
- D25 pad 1: R2 -> R1
- D26 pad 1: R2 -> R1
- D27 pad 1: R2 -> R1
- D28 pad 1: R2 -> R4
- D3 pad 1: R1 -> R0
- D33 pad 1: R3 -> R2
- D34 pad 1: R3 -> R2
- D35 pad 1: R3 -> R2
- D36 pad 1: R3 -> R2
- D37 pad 1: R3 -> R2
- D38 pad 1: R3 -> R2
- D39 pad 1: R3 -> R2
- D4 pad 1: R1 -> R0
- D40 pad 1: R3 -> R2
- D41 pad 1: R3 -> R2
- D42 pad 1: R3 -> R4
- D48 pad 1: R4 -> R3
- D49 pad 1: R4 -> R3
- D5 pad 1: R1 -> R0
- D50 pad 1: R4 -> R3
- D51 pad 1: R4 -> R3
- D52 pad 1: R4 -> R3
- D53 pad 1: R4 -> R3
- D54 pad 1: R4 -> R3
- D55 pad 1: R4 -> R5
- D6 pad 1: R1 -> R0
- D62 pad 1: R5 -> R4
- D63 pad 1: R5 -> R4
- D64 pad 1: R5 -> R4
- D65 pad 1: R5 -> R4
- D66 pad 1: R5 -> R4
- D7 pad 1: R1 -> R0
- D75 pad 1: R6 -> R5
- D76 pad 1: R6 -> R5
- D8 pad 1: R1 -> R0
- D9 pad 1: R1 -> R0
- S1 pad 1: C1 -> C0
- S10 pad 1: C10 -> C9
- S11 pad 1: C11 -> C10
- S12 pad 1: C12 -> C11
- S13 pad 1: C13 -> C12
- S14 pad 1: C14 -> C12
- S15 pad 1: C15 -> C0
- S16 pad 1: C16 -> C1
- S17 pad 1: C1 -> C2
- S18 pad 1: C2 -> C3
- S19 pad 1: C3 -> C4
- S2 pad 1: C2 -> C1
- S20 pad 1: C4 -> C5
- S21 pad 1: C5 -> C6
- S22 pad 1: C6 -> C7
- S23 pad 1: C7 -> C8
- S24 pad 1: C8 -> C9
- S25 pad 1: C9 -> C10
- S26 pad 1: C10 -> C11
- S27 pad 1: C11 -> C12
- S28 pad 1: C12 -> C11
- S29 pad 1: C13 -> C0
- S3 pad 1: C3 -> C2
- S30 pad 1: C14 -> C1
- S31 pad 1: C15 -> C2
- S32 pad 1: C16 -> C3
- S33 pad 1: C1 -> C4
- S34 pad 1: C2 -> C5
- S35 pad 1: C3 -> C6
- S36 pad 1: C4 -> C7
- S37 pad 1: C5 -> C8
- S38 pad 1: C6 -> C9
- S39 pad 1: C7 -> C10
- S4 pad 1: C4 -> C3
- S40 pad 1: C8 -> C11
- S41 pad 1: C9 -> C12
- S42 pad 1: C10 -> C12
- S43 pad 1: C11 -> C0
- S44 pad 1: C12 -> C1
- S45 pad 1: C13 -> C2
- S46 pad 1: C14 -> C3
- S47 pad 1: C15 -> C4
- S48 pad 1: C1 -> C5
- S49 pad 1: C2 -> C6
- S5 pad 1: C5 -> C4
- S50 pad 1: C3 -> C7
- S51 pad 1: C4 -> C8
- S52 pad 1: C5 -> C9
- S53 pad 1: C6 -> C10
- S54 pad 1: C7 -> C11
- S55 pad 1: C8 -> C9
- S56 pad 1: C9 -> C0
- S57 pad 1: C10 -> C1
- S58 pad 1: C11 -> C2
- S59 pad 1: C12 -> C3
- S6 pad 1: C6 -> C5
- S60 pad 1: C14 -> C4
- S61 pad 1: C15 -> C5
- S62 pad 1: C1 -> C6
- S63 pad 1: C2 -> C7
- S64 pad 1: C3 -> C8
- S65 pad 1: C4 -> C9
- S66 pad 1: C5 -> C10
- S67 pad 1: C6 -> C10
- S68 pad 1: C7 -> C0
- S69 pad 1: C8 -> C1
- S7 pad 1: C7 -> C6
- S70 pad 1: C9 -> C2
- S71 pad 1: C10 -> C3
- S72 pad 1: C11 -> C4
- S73 pad 1: C14 -> C5
- S74 pad 1: C15 -> C6
- S75 pad 1: C1 -> C7
- S76 pad 1: C2 -> C8
- S8 pad 1: C8 -> C7
- S9 pad 1: C9 -> C8
- U1 pad 1: R6 -> C0
- U1 pad 10: C15 -> C7
- U1 pad 11: R1 -> C8
- U1 pad 12: C8 -> C9
- U1 pad 14: C9 -> C10
- U1 pad 15: C10 -> C11
- U1 pad 16: C11 -> C12
- U1 pad 17: C12 -> R0
- U1 pad 19: C13 -> R1
- U1 pad 2: R5 -> C1
- U1 pad 20: C14 -> R2
- U1 pad 21: C7 -> R3
- U1 pad 22: C6 -> R4
- U1 pad 24: C5 -> R5
- U1 pad 25: C4 -> unconnected-(U1-GPIO19-Pad25)
- U1 pad 26: C3 -> unconnected-(U1-GPIO20-Pad26)
- U1 pad 27: C2 -> unconnected-(U1-GPIO21-Pad27)
- U1 pad 29: C1 -> unconnected-(U1-GPIO22-Pad29)
- U1 pad 4: R4 -> C2
- U1 pad 5: R3 -> C3
- U1 pad 6: R2 -> C4
- U1 pad 7: C17 -> C5
- U1 pad 9: C16 -> C6
Routing:
- net R6: track 320.2 -> 0.00 mm
- net R2: track 313.9 -> 0.00 mm
- net R1: track 309.6 -> 0.00 mm
- net R5: track 301.1 -> 0.00 mm
- net R4: track 294.8 -> 0.00 mm
- net R3: track 290.5 -> 0.00 mm
- net C10: track 147.5 -> 0.00 mm
- net C9: track 146.2 -> 0.00 mm
- net C8: track 146.2 -> 0.00 mm
- net C11: track 146.1 -> 0.00 mm
- net C14: track 144.9 -> 0.00 mm
- net C2: track 137.8 -> 0.00 mm
- net C5: track 136.4 -> 0.00 mm
- net C3: track 135.9 -> 0.00 mm
- net C1: track 133.9 -> 0.00 mm
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Other:
- board outline removed

Commit message: Complete wiring
Parts:
- moved D76 206.2 mm to (342.9, 192.9)
- moved D75 199.6 mm to (323.9, 192.9)
- moved D74 193.5 mm to (304.8, 192.9)
- moved D68 191.2 mm to (78.6, 192.9)
- moved D73 188.0 mm to (285.8, 192.9)
- moved D69 184.0 mm to (102.4, 192.9)
- moved D72 183.1 mm to (266.7, 192.9)
- moved D70 178.1 mm to (126.2, 192.9)
- moved D67 173.4 mm to (326.2, 173.8)
- moved D71 169.3 mm to (197.6, 192.9)
- moved D55 164.1 mm to (331.0, 154.8)
- moved D56 163.6 mm to (88.1, 173.8)
- moved D57 153.5 mm to (119.1, 173.8)
- moved D66 151.8 mm to (290.5, 173.8)
- moved D58 149.5 mm to (138.1, 173.8)
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Connections:
- U1 pad 21: R3 -> R5
- U1 pad 24: R5 -> R3
Routing:
- net R5: track 0.00 -> 643.0 mm
- net R4: track 0.00 -> 575.6 mm
- net R3: track 0.00 -> 556.5 mm
- net R2: track 0.00 -> 484.1 mm
- net R1: track 0.00 -> 472.3 mm
- net R0: track 0.00 -> 453.1 mm
- net C9: track 0.00 -> 334.0 mm
- net C8: track 0.00 -> 327.5 mm
- net C12: track 0.00 -> 318.5 mm
- net C7: track 0.00 -> 310.9 mm
- net C11: track 0.00 -> 304.2 mm
- net C10: track 0.00 -> 302.9 mm
- net C6: track 0.00 -> 294.3 mm
- net C5: track 0.00 -> 284.0 mm
- net C4: track 0.00 -> 256.8 mm
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
Commit message: Change layout
Parts:
- added D77: Diode, ScottoKeebs_Components:Diode_SOD-123, B.Cu at (342.9, 97.6)
- added S77: Del, ScottoKeebs_MX:MX_Plate_1.00u, F.Cu at (333.4, 104.8)
- S1, S10, S11, S12, S13, S15, S16, S17, S18, S19, S2, S20, S21, S22, S23, S24, S25, S26, S27, S3, S30, S31, S32, S33, S34, S35, S36, S37, S38, S39, S4, S40, S41, S44, S45, S46, S47, S48, S49, S5, S50, S51, S52, S53, S54, S57, S58, S59, S6, S60, S61, S62, S63, S64, S65, S66, S7, S73, S74, S75, S76, S8, S9: footprint ScottoKeebs_MX:MX_PCB_1.00u -> ScottoKeebs_MX:MX_Plate_1.00u
- S14: value Del -> Print; footprint ScottoKeebs_MX:MX_PCB_1.00u -> ScottoKeebs_MX:MX_Plate_1.00u
- S28: footprint ScottoKeebs_MX:MX_PCB_2.00u -> ScottoKeebs_MX:MX_Plate_2.00u
- S29, S42: footprint ScottoKeebs_MX:MX_PCB_1.50u -> ScottoKeebs_MX:MX_Plate_1.50u
- S43: footprint ScottoKeebs_MX:MX_PCB_1.75u -> ScottoKeebs_MX:MX_Plate_1.75u
- S55, S56: footprint ScottoKeebs_MX:MX_PCB_2.25u -> ScottoKeebs_MX:MX_Plate_2.25u
- S67: footprint ScottoKeebs_MX:MX_PCB_2.75u -> ScottoKeebs_MX:MX_Plate_2.75u
- S68, S69, S70: footprint ScottoKeebs_MX:MX_PCB_1.25u -> ScottoKeebs_MX:MX_Plate_1.25u
- S71: value Space -> Fn; footprint ScottoKeebs_MX:MX_PCB_6.25u -> ScottoKeebs_MX:MX_Plate_1.00u
- S72: value Fn -> Space; footprint ScottoKeebs_MX:MX_PCB_1.00u -> ScottoKeebs_MX:MX_Plate_6.25u
- moved U1 95.6 mm to (195.3, 79.8)
- moved D71 50.0 mm to (147.6, 192.9)
- moved S72 50.0 mm to (207.2, 200.0)
- moved S71 50.0 mm to (138.1, 200.0)
- moved D72 46.4 mm to (220.3, 192.9)
- moved S14 19.6 mm to (314.3, 104.8)
- moved D14 19.6 mm to (323.9, 97.6)
- moved S13 15.1 mm to (295.3, 104.8)
- moved D11 15.1 mm to (266.7, 97.6)
- moved D12 15.1 mm to (285.8, 97.6)
- moved S10 15.1 mm to (238.1, 104.8)
- moved D10 15.1 mm to (247.7, 97.6)
- moved S11 15.1 mm to (257.2, 104.8)
- moved S12 15.1 mm to (276.2, 104.8)
- moved D13 15.1 mm to (304.8, 97.6)
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Connections:
- D14 pad 1: R3 -> R5
- D28 pad 1: R4 -> R5
- D42 pad 1: R4 -> R3
- D55 pad 1: R5 -> R4
- D67 pad 1: R5 -> R4
- S14 pad 1: C12 -> C9
- S55 pad 1: C9 -> C12
- S67 pad 1: C10 -> C11
- U1 pad 21: R5 -> R4
- U1 pad 22: R4 -> R3
- U1 pad 24: R3 -> R5
Routing:
- net C12: track 318.5 -> 188.5 mm
- net C9: track 334.0 -> 217.4 mm
- net R4: track 575.6 -> 470.3 mm
- net R0: track 453.1 -> 349.6 mm
- net C8: track 327.5 -> 226.4 mm
- net C7: track 310.9 -> 210.4 mm
- net R3: track 556.5 -> 460.3 mm
- net C0: track 132.5 -> 222.5 mm
- net C1: track 140.4 -> 219.3 mm
- net C6: track 294.3 -> 218.1 mm
- net C10: track 302.9 -> 233.4 mm
- net R5: track 643.0 -> 709.2 mm
- net C4: track 256.8 -> 194.4 mm
- net C2: track 153.3 -> 202.7 mm
- net C5: track 284.0 -> 235.7 mm
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Other:
- board outline added: 295.3 x 152.4 mm

Commit message: Add Usb C header and XH 2.54 header
Parts:
- added J1: USB_C_Receptacle_USB2.0_14P, Connector_USB:USB_C_Receptacle_GCT_USB4085, F.Cu at (70.1, 71.0)
- added J2: Conn_01x04_Socket, Connector_PinHeader_2.54mm:PinHeader_1x04_P2.54mm_Vertical, F.Cu at (100.0, 73.3)
- added R1: 5.1k, Resistor_SMD:R_0612_1632Metric_Pad1.18x3.40mm_HandSolder, F.Cu at (76.2, 69.1)
- added R2: 5.1k, Resistor_SMD:R_0612_1632Metric_Pad1.18x3.40mm_HandSolder, F.Cu at (81.0, 69.1)
- renumbered S44 to A, S27 to Add, S70 to Alt, S61 to B, S28 to Backspace, S15 to Backtick, S59 to C, S43 to Caps, S64 to Comma, S68 to Ctrl, S73 to Custom_1, S74 to Custom_2, S75 to Custom_3, S76 to Custom_4, S46 to D, S77 to Del, S32 to E, S55 to Enter, S1 to Esc, S47 to F, S2 to F1, S11 to F10, S12 to F11, S13 to F12, S3 to F2, S4 to F3, S5 to F4, S6 to F5, S7 to F6, S8 to F7, S9 to F8, S10 to F9, S71 to Fn, S48 to G, S49 to H, S37 to I, S50 to J, S51 to K, S52 to L, S56 to L.Shift, S40 to L.Sqr, S63 to M, S26 to Minus, S62 to N, S25 to Num_0, S16 to Num_1, S17 to Num_2, S18 to Num_3, S19 to Num_4, S20 to Num_5, S21 to Num_6, S22 to Num_7, S23 to Num_8, S24 to Num_9, S38 to O, S39 to P, S42 to Pipe, S14 to Print, S65 to Priod, S30 to Q, S54 to Quote, S33 to R, S67 to R.Shift, S41 to R.Sqr, S45 to S, S53 to Semi, S66 to Slash, S72 to Space, S69 to Super, S34 to T, S29 to Tab, S36 to U, S60 to V, S31 to W, S58 to X, S35 to Y, S57 to Z
Routing:
- net GND: track 0.00 -> 83.5 mm
- net Net-(J2-Pin_1): track 0.00 -> 39.8 mm
- net D-: track 0.00 -> 38.4 mm
- net D+: track 0.00 -> 36.5 mm
- net Net-(J1-CC2): track 0.00 -> 16.8 mm
- net Net-(J1-CC1): track 0.00 -> 12.5 mm, vias 0 -> 2
- net C12: track 188.5 -> 191.0 mm
- net C6: track 218.1 -> 216.9 mm
- added copper zone on B.Cu, net (none)
- added copper zone on F.Cu, net (none)

Commit message: Fix
Parts:
- R1, R2: footprint Resistor_SMD:R_0612_1632Metric_Pad1.18x3.40mm_HandSolder -> Resistor_SMD:R_0201_0603Metric_Pad0.64x0.40mm_HandSolder; moved to B.Cu
- S1: renamed from Esc; footprint ScottoKeebs_MX:MX_Plate_1.00u -> ScottoKeebs_MX:MX_PCB_1.00u
- S10: renamed from F9; footprint ScottoKeebs_MX:MX_Plate_1.00u -> ScottoKeebs_MX:MX_PCB_1.00u
- S11: renamed from F10; footprint ScottoKeebs_MX:MX_Plate_1.00u -> ScottoKeebs_MX:MX_PCB_1.00u
- S12: renamed from F11; footprint ScottoKeebs_MX:MX_Plate_1.00u -> ScottoKeebs_MX:MX_PCB_1.00u
- S13: renamed from F12; footprint ScottoKeebs_MX:MX_Plate_1.00u -> ScottoKeebs_MX:MX_PCB_1.00u
- S14: renamed from Print; footprint ScottoKeebs_MX:MX_Plate_1.00u -> ScottoKeebs_MX:MX_PCB_1.00u
- S15: renamed from Backtick; footprint ScottoKeebs_MX:MX_Plate_1.00u -> ScottoKeebs_MX:MX_PCB_1.00u
- S16: renamed from Num_1; footprint ScottoKeebs_MX:MX_Plate_1.00u -> ScottoKeebs_MX:MX_PCB_1.00u
- S17: renamed from Num_2; footprint ScottoKeebs_MX:MX_Plate_1.00u -> ScottoKeebs_MX:MX_PCB_1.00u
- S18: renamed from Num_3; footprint ScottoKeebs_MX:MX_Plate_1.00u -> ScottoKeebs_MX:MX_PCB_1.00u
- S19: renamed from Num_4; footprint ScottoKeebs_MX:MX_Plate_1.00u -> ScottoKeebs_MX:MX_PCB_1.00u
- S2: renamed from F1; footprint ScottoKeebs_MX:MX_Plate_1.00u -> ScottoKeebs_MX:MX_PCB_1.00u
- S20: renamed from Num_5; footprint ScottoKeebs_MX:MX_Plate_1.00u -> ScottoKeebs_MX:MX_PCB_1.00u
- S21: renamed from Num_6; footprint ScottoKeebs_MX:MX_Plate_1.00u -> ScottoKeebs_MX:MX_PCB_1.00u
- S22: renamed from Num_7; footprint ScottoKeebs_MX:MX_Plate_1.00u -> ScottoKeebs_MX:MX_PCB_1.00u
- S23: renamed from Num_8; footprint ScottoKeebs_MX:MX_Plate_1.00u -> ScottoKeebs_MX:MX_PCB_1.00u
- S24: renamed from Num_9; footprint ScottoKeebs_MX:MX_Plate_1.00u -> ScottoKeebs_MX:MX_PCB_1.00u
- S25: renamed from Num_0; footprint ScottoKeebs_MX:MX_Plate_1.00u -> ScottoKeebs_MX:MX_PCB_1.00u
- S26: renamed from Minus; footprint ScottoKeebs_MX:MX_Plate_1.00u -> ScottoKeebs_MX:MX_PCB_1.00u
- S27: renamed from Add; footprint ScottoKeebs_MX:MX_Plate_1.00u -> ScottoKeebs_MX:MX_PCB_1.00u
- S28: renamed from Backspace; footprint ScottoKeebs_MX:MX_Plate_2.00u -> ScottoKeebs_MX:MX_PCB_2.00u
- S29: renamed from Tab; footprint ScottoKeebs_MX:MX_Plate_1.50u -> ScottoKeebs_MX:MX_PCB_1.50u
- S3: renamed from F2; footprint ScottoKeebs_MX:MX_Plate_1.00u -> ScottoKeebs_MX:MX_PCB_1.00u
- S30: renamed from Q; footprint ScottoKeebs_MX:MX_Plate_1.00u -> ScottoKeebs_MX:MX_PCB_1.00u
- S31: renamed from W; footprint ScottoKeebs_MX:MX_Plate_1.00u -> ScottoKeebs_MX:MX_PCB_1.00u
- S32: renamed from E; footprint ScottoKeebs_MX:MX_Plate_1.00u -> ScottoKeebs_MX:MX_PCB_1.00u
- S33: renamed from R; footprint ScottoKeebs_MX:MX_Plate_1.00u -> ScottoKeebs_MX:MX_PCB_1.00u
- S34: renamed from T; footprint ScottoKeebs_MX:MX_Plate_1.00u -> ScottoKeebs_MX:MX_PCB_1.00u
- S35: renamed from Y; footprint ScottoKeebs_MX:MX_Plate_1.00u -> ScottoKeebs_MX:MX_PCB_1.00u
- S36: renamed from U; footprint ScottoKeebs_MX:MX_Plate_1.00u -> ScottoKeebs_MX:MX_PCB_1.00u
- S37: renamed from I; footprint ScottoKeebs_MX:MX_Plate_1.00u -> ScottoKeebs_MX:MX_PCB_1.00u
- S38: renamed from O; footprint ScottoKeebs_MX:MX_Plate_1.00u -> ScottoKeebs_MX:MX_PCB_1.00u
- S39: renamed from P; footprint ScottoKeebs_MX:MX_Plate_1.00u -> ScottoKeebs_MX:MX_PCB_1.00u
- S4: renamed from F3; footprint ScottoKeebs_MX:MX_Plate_1.00u -> ScottoKeebs_MX:MX_PCB_1.00u
- S40: renamed from L.Sqr; footprint ScottoKeebs_MX:MX_Plate_1.00u -> ScottoKeebs_MX:MX_PCB_1.00u
- S41: renamed from R.Sqr; footprint ScottoKeebs_MX:MX_Plate_1.00u -> ScottoKeebs_MX:MX_PCB_1.00u
- S42: renamed from Pipe; footprint ScottoKeebs_MX:MX_Plate_1.50u -> ScottoKeebs_MX:MX_PCB_1.50u
- S43: renamed from Caps; footprint ScottoKeebs_MX:MX_Plate_1.75u -> ScottoKeebs_MX:MX_PCB_1.75u
- S44: renamed from A; footprint ScottoKeebs_MX:MX_Plate_1.00u -> ScottoKeebs_MX:MX_PCB_1.00u
- S45: renamed from S; footprint ScottoKeebs_MX:MX_Plate_1.00u -> ScottoKeebs_MX:MX_PCB_1.00u
- S46: renamed from D; footprint ScottoKeebs_MX:MX_Plate_1.00u -> ScottoKeebs_MX:MX_PCB_1.00u
- S47: renamed from F; footprint ScottoKeebs_MX:MX_Plate_1.00u -> ScottoKeebs_MX:MX_PCB_1.00u
- S48: renamed from G; footprint ScottoKeebs_MX:MX_Plate_1.00u -> ScottoKeebs_MX:MX_PCB_1.00u
- S49: renamed from H; footprint ScottoKeebs_MX:MX_Plate_1.00u -> ScottoKeebs_MX:MX_PCB_1.00u
- S5: renamed from F4; footprint ScottoKeebs_MX:MX_Plate_1.00u -> ScottoKeebs_MX:MX_PCB_1.00u
- S50: renamed from J; footprint ScottoKeebs_MX:MX_Plate_1.00u -> ScottoKeebs_MX:MX_PCB_1.00u
- S51: renamed from K; footprint ScottoKeebs_MX:MX_Plate_1.00u -> ScottoKeebs_MX:MX_PCB_1.00u
- S52: renamed from L; footprint ScottoKeebs_MX:MX_Plate_1.00u -> ScottoKeebs_MX:MX_PCB_1.00u
- S53: renamed from Semi; footprint ScottoKeebs_MX:MX_Plate_1.00u -> ScottoKeebs_MX:MX_PCB_1.00u
- S54: renamed from Quote; footprint ScottoKeebs_MX:MX_Plate_1.00u -> ScottoKeebs_MX:MX_PCB_1.00u
- S55: renamed from Enter; footprint ScottoKeebs_MX:MX_Plate_2.25u -> ScottoKeebs_MX:MX_PCB_2.25u
- S56: renamed from L.Shift; footprint ScottoKeebs_MX:MX_Plate_2.25u -> ScottoKeebs_MX:MX_PCB_2.25u
- S57: renamed from Z; footprint ScottoKeebs_MX:MX_Plate_1.00u -> ScottoKeebs_MX:MX_PCB_1.00u
- S58: renamed from X; footprint ScottoKeebs_MX:MX_Plate_1.00u -> ScottoKeebs_MX:MX_PCB_1.00u
- S59: renamed from C; footprint ScottoKeebs_MX:MX_Plate_1.00u -> ScottoKeebs_MX:MX_PCB_1.00u
- S6: renamed from F5; footprint ScottoKeebs_MX:MX_Plate_1.00u -> ScottoKeebs_MX:MX_PCB_1.00u
- S60: renamed from V; footprint ScottoKeebs_MX:MX_Plate_1.00u -> ScottoKeebs_MX:MX_PCB_1.00u
- S61: renamed from B; footprint ScottoKeebs_MX:MX_Plate_1.00u -> ScottoKeebs_MX:MX_PCB_1.00u
- S62: renamed from N; footprint ScottoKeebs_MX:MX_Plate_1.00u -> ScottoKeebs_MX:MX_PCB_1.00u
- S63: renamed from M; footprint ScottoKeebs_MX:MX_Plate_1.00u -> ScottoKeebs_MX:MX_PCB_1.00u
- S64: renamed from Comma; footprint ScottoKeebs_MX:MX_Plate_1.00u -> ScottoKeebs_MX:MX_PCB_1.00u
- S65: renamed from Priod; footprint ScottoKeebs_MX:MX_Plate_1.00u -> ScottoKeebs_MX:MX_PCB_1.00u
- S66: renamed from Slash; footprint ScottoKeebs_MX:MX_Plate_1.00u -> ScottoKeebs_MX:MX_PCB_1.00u
- S67: renamed from R.Shift; footprint ScottoKeebs_MX:MX_Plate_2.75u -> ScottoKeebs_MX:MX_PCB_2.75u
- S68: renamed from Ctrl; footprint ScottoKeebs_MX:MX_Plate_1.25u -> ScottoKeebs_MX:MX_PCB_1.25u
- S69: renamed from Super; footprint ScottoKeebs_MX:MX_Plate_1.25u -> ScottoKeebs_MX:MX_PCB_1.25u
- S7: renamed from F6; footprint ScottoKeebs_MX:MX_Plate_1.00u -> ScottoKeebs_MX:MX_PCB_1.00u
- S70: renamed from Alt; footprint ScottoKeebs_MX:MX_Plate_1.25u -> ScottoKeebs_MX:MX_PCB_1.25u
- S71: renamed from Fn; footprint ScottoKeebs_MX:MX_Plate_1.00u -> ScottoKeebs_MX:MX_PCB_1.00u
- S72: renamed from Space; footprint ScottoKeebs_MX:MX_Plate_6.25u -> ScottoKeebs_MX:MX_PCB_6.25u
- S73: renamed from Custom_1; footprint ScottoKeebs_MX:MX_Plate_1.00u -> ScottoKeebs_MX:MX_PCB_1.00u
- S74: renamed from Custom_2; footprint ScottoKeebs_MX:MX_Plate_1.00u -> ScottoKeebs_MX:MX_PCB_1.00u
- S75: renamed from Custom_3; footprint ScottoKeebs_MX:MX_Plate_1.00u -> ScottoKeebs_MX:MX_PCB_1.00u
- S76: renamed from Custom_4; footprint ScottoKeebs_MX:MX_Plate_1.00u -> ScottoKeebs_MX:MX_PCB_1.00u
- S77: renamed from Del; footprint ScottoKeebs_MX:MX_Plate_1.00u -> ScottoKeebs_MX:MX_PCB_1.00u
- S8: renamed from F7; footprint ScottoKeebs_MX:MX_Plate_1.00u -> ScottoKeebs_MX:MX_PCB_1.00u
- S9: renamed from F8; footprint ScottoKeebs_MX:MX_Plate_1.00u -> ScottoKeebs_MX:MX_PCB_1.00u
- moved R2 7.53 mm to (73.8, 71.4), turned to -90 degrees
- moved R1 2.38 mm to (76.2, 71.4), turned to 90 degrees
Routing:
- net GND: track 83.5 -> 70.9 mm
- net C11: track 263.5 -> 272.4 mm
- net Net-(J1-CC2): track 16.8 -> 10.0 mm
- net Net-(J1-CC1): track 12.5 -> 8.95 mm, vias 2 -> 0
- net C0: track 222.5 -> 225.3 mm
- net C3: track 184.7 -> 186.3 mm
- net C12: track 191.0 -> 189.7 mm
- net C2: track 202.7 -> 203.8 mm
