File: PCB/PicoKeyboard/PicoKeyboard.kicad_pcb (KiCad board)
At the start: 2 copper layers, 295.3 x 152.4 mm, 159 parts, among them J1 USB_C_Receptacle_USB2.0_14P, J2 Conn_01x04_Socket, U1 Raspberry_Pi_Pico

Commit message: Rewired
Routing:
- net C4: track 194.6 -> 211.6 mm
- net C11: track 272.4 -> 258.0 mm
- net C0: track 225.3 -> 238.9 mm
- net C7: track 210.6 -> 223.8 mm
- net C6: track 217.1 -> 230.2 mm
- net C8: track 226.6 -> 239.7 mm
- net C9: track 217.7 -> 229.7 mm
- net C3: track 186.3 -> 197.9 mm
- net C2: track 203.8 -> 215.3 mm
- net C1: track 219.5 -> 230.6 mm
- net C10: track 233.6 -> 243.8 mm
- net C5: track 235.9 -> 245.0 mm
- net R5: track 709.2 -> 707.6 mm
- net C12: track 189.7 -> 188.6 mm
- net D-: track 38.4 -> 39.3 mm
- removed copper zone on B.Cu, net (none)
- removed copper zone on F.Cu, net (none)

Commit message: Change gpio pin
Connections:
- U1 pad 21: R4 -> unconnected-(U1-GPIO16-Pad21)
- U1 pad 22: R3 -> unconnected-(U1-GPIO17-Pad22)
- U1 pad 24: R5 -> R4
- U1 pad 25: unconnected-(U1-GPIO19-Pad25) -> R3
- U1 pad 26: unconnected-(U1-GPIO20-Pad26) -> R5
Routing:
- net R0: track 349.6 -> 368.7 mm
- net Net-(J1-CC1): track 8.95 -> 12.6 mm
- net R3: track 460.3 -> 463.5 mm
- net R5: track 707.6 -> 708.8 mm
- net GND: track 71.3 -> 72.3 mm
- net C8: track 239.7 -> 238.7 mm
- net R2: track 457.8 -> 458.7 mm
- net C9: track 229.7 -> 229.2 mm
- net D+: track 36.8 -> 37.4 mm
- net C2: track 215.3 -> 214.8 mm
- added copper zone on B.Cu, net (none)
- added copper zone on F.Cu, net (none)
