File: PCB/PicoKeyboard/PicoKeyboard.kicad_pcb (KiCad board)
At the start: 2 copper layers, 295.3 x 152.4 mm, 162 parts, among them J1 USB_C_Receptacle_USB2.0_14P, J2 Conn_01x04_Socket, J3 Conn_01x04_Socket, U1 Raspberry_Pi_Pico

Commit message: Add firmware
Parts:
- C1: value 100nF -> C_Small
- C2: value 1uF -> C_Small
- S27: value Add -> Equals
Changed lines of the file:
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@@
 			)
 		)
-		(property "Value" "Add"
+		(property "Value" "Equals"
 			(at 0 8 0)
 			(layer "F.Fab")
@@
 		)
 		(fp_text user "SWCLK"
-			(at -2.54 20.25 360)
+			(at -2.54 20.25 0)
 			(layer "F.SilkS")
 			(effects
@@
 		)
 		(fp_text user "GND"
-			(at 0 21 360)
+			(at 0 21 0)
 			(layer "F.SilkS")
 			(effects
@@
 		)
 		(fp_text user "SWDIO"
-			(at 2.54 20.25 360)
+			(at 2.54 20.25 0)
 			(layer "F.SilkS")
 			(effects
@@
 			)
 		)
-		(property "Value" "100nF"
+		(property "Value" "C_Small"
 			(at 1.969375 0 180)
 			(layer "B.SilkS")
@@
 			)
 		)
-		(property "Value" "1uF"
+		(property "Value" "C_Small"
 			(at 1.869375 0 180)
 			(layer "B.SilkS")

Commit message: Update PCB
Parts:
- C1: value C_Small -> 100nF
- C2: value C_Small -> 1uF
- S15: value Backtick -> Tilde
- S40: value [ -> LBrace
- S41: value ] -> RBrace
- S42: value Pipe -> BSlash
- S56: value L.Shift -> LShift
- S67: value R.Shift -> RShift
Routing:
- net R4: track 601.3 -> 606.7 mm
- net C8: track 702.4 -> 706.8 mm
- net C10: track 370.6 -> 373.9 mm
- net C6: track 586.8 -> 583.9 mm
- net C1: track 276.4 -> 279.3 mm
- net R2: track 504.1 -> 501.5 mm
- net R5: track 531.5 -> 533.6 mm
- net R3: track 419.1 -> 417.3 mm
- net C7: track 484.4 -> 485.9 mm
- net C5: track 1046.7 -> 1047.7 mm
- net C9: track 530.3 -> 531.2 mm
- net C3: track 606.3 -> 606.8 mm
Other:
- board text added: "01 x Raspberry Pico (RP2040) 77 x Hotswap socket (Kailh) 77 x Diode T4 SOD-123 (1N4148W SMD1206) 01 x USB-C Receptacle (USB4085) 01 x Pin header (XH2.54 4 pins) 01 x Pin socket (XH2.54 4 pins) 02 x Resistor SMD-0603 (5.1k Ohm) 01 x Capacitor SMD-0603 (100nF) 01 x Capacitor SMD-0603 (1uF) 01 x 0.96in OLED (SSD1315 White)"
- board text removed: "01 x Raspberry Pico (RP2040) 77 x Hotswap socket (Kailh) 77 x Diode T4 SOD-123 (1N4148W SMD1206) 01 x USB-C Receptacle (USB4085) 01 x Pin header (XH2.54 4 pins) 01 x Pin socket (XH2.54 4 pins) 02 x Resistor SMD-0603 (5.1k Ohm) 01 x Capacitor SMD-0603 (100nF) 01 x Capacitor SMD-0603 (1uF)"

Commit message: Update PCB
Parts:
- added C3: 1uF, Capacitor_SMD:C_0201_0603Metric_Pad0.64x0.40mm_HandSolder, B.Cu at (90.5, 81.5)
- added C4: 100nF, Capacitor_SMD:C_0201_0603Metric_Pad0.64x0.40mm_HandSolder, B.Cu at (95.5, 81.5)
- J2: value Conn_01x04_Socket -> XH2.54 Socket 1x04
- J3: value Conn_01x04_Socket -> Header 4 pins
- moved R1 2.50 mm to (80.0, 70.0)
- turned R2 to 90 degrees
Connections:
- J1 pad A4: Net-(J2-Pin_1) -> VCC
- J1 pad A9: Net-(J2-Pin_1) -> VCC
- J1 pad B4: Net-(J2-Pin_1) -> VCC
- J1 pad B9: Net-(J2-Pin_1) -> VCC
- J2 pad 1: Net-(J2-Pin_1) -> GND
- J2 pad 4: GND -> VCC
Routing:
- net VCC: track 0.00 -> 52.1 mm
- net Net-(J2-Pin_1): track 40.9 -> 0.00 mm
- net GND: track 80.2 -> 100.0 mm
- net Net-(J1-CC1): track 19.7 -> 16.0 mm, vias 2 -> 0
- net Net-(D76-A): track 13.7 -> 12.1 mm
- net R0: track 267.2 -> 268.4 mm
- net C9: track 531.2 -> 532.2 mm
- net R4: track 606.7 -> 607.6 mm
- net Net-(J1-CC2): track 11.4 -> 12.1 mm
- net D-: track 40.8 -> 41.4 mm
- net R2: track 501.5 -> 502.1 mm
Other:
- board text added: "01 x Raspberry Pico (RP2040) 77 x Hotswap socket (Kailh) 77 x Diode T4 SOD-123 (1N4148W SMD1206) 01 x USB-C Receptacle (USB4085) 01 x Pins header (4 pins) 01 x Pin socket (XH2.54 1x04) 02 x Resistor SMD-0603 (5.1k Ohm) 02 x Capacitor SMD-0603 (100nF) 02 x Capacitor SMD-0603 (1uF) 01 x 0.96in OLED (SSD1315 White)"
- board text added: "https://github.com/lulkien"
- board text removed: "01 x Raspberry Pico (RP2040) 77 x Hotswap socket (Kailh) 77 x Diode T4 SOD-123 (1N4148W SMD1206) 01 x USB-C Receptacle (USB4085) 01 x Pin header (XH2.54 4 pins) 01 x Pin socket (XH2.54 4 pins) 02 x Resistor SMD-0603 (5.1k Ohm) 01 x Capacitor SMD-0603 (100nF) 01 x Capacitor SMD-0603 (1uF) 01 x 0.96in OLED (SSD1315 White)"
