File: PCB/PicoKeyboard/PicoKeyboard.kicad_pcb (KiCad board)
At the start: 2 copper layers, 295.3 x 152.4 mm, 164 parts, among them J1 USB_C_Receptacle_USB2.0_14P, J2 XH2.54 Socket 1x04, J3 Header 4 pins, U1 Raspberry_Pi_Pico

Commit message: Update PCB
Parts:
- J1: footprint Connector_USB:USB_C_Receptacle_GCT_USB4085 -> Connector_USB:USB_C_Receptacle_GCT_USB4110
- J2: value XH2.54 Socket 1x04 -> Conn_01x04_Socket
- J3: value Header 4 pins -> Conn_01x04_Socket
- moved R1 8.73 mm to (88.0, 73.5), turned to -90 degrees
- moved J1 6.23 mm to (67.0, 65.6)
- moved R2 6.10 mm to (81.0, 73.5), turned to -90 degrees
- moved C3 2.45 mm to (88.1, 81.0)
- moved C4 1.54 mm to (94.1, 81.0)
Routing:
- net D-: track 41.4 -> 48.5 mm
- net Net-(J1-CC2): track 12.1 -> 19.1 mm, vias 0 -> 1
- net Net-(J1-CC1): track 16.0 -> 22.8 mm, vias 0 -> 1
- net GND: track 100.0 -> 105.3 mm, vias 0 -> 1
- net (no net): track 0.00 -> 4.81 mm
- net D+: track 37.9 -> 40.9 mm, vias 0 -> 1
- net VCC: vias 0 -> 1
Other:
- board text added: "01 x Raspberry Pico (RP2040) 77 x Hotswap socket (Kailh) 77 x Diode T4 SOD-123 (1N4148W SMD1206) 01 x USB-C Receptacle (USB4110) 02 x Pin socket (XH2.54 1x04) 02 x Resistor SMD-0603 (5.1k Ohm) 02 x Capacitor SMD-0603 (100nF) 02 x Capacitor SMD-0603 (1uF) 01 x 0.96in OLED (SSD1315 White)"
- board text removed: "01 x Raspberry Pico (RP2040) 77 x Hotswap socket (Kailh) 77 x Diode T4 SOD-123 (1N4148W SMD1206) 01 x USB-C Receptacle (USB4085) 01 x Pins header (4 pins) 01 x Pin socket (XH2.54 1x04) 02 x Resistor SMD-0603 (5.1k Ohm) 02 x Capacitor SMD-0603 (100nF) 02 x Capacitor SMD-0603 (1uF) 01 x 0.96in OLED (SSD1315 White)"

Commit message: Update design
Parts:
- moved R2 11.0 mm to (92.0, 73.5)
- moved J1 9.92 mm to (76.9, 65.6)
Connections:
- J2 pad 2: D+ -> D-
- J2 pad 3: D- -> D+
Routing:
- net D-: track 48.5 -> 30.1 mm, vias 0 -> 1
- net Net-(J1-CC1): track 22.8 -> 11.8 mm
- net VCC: track 52.1 -> 42.3 mm
- net D+: track 40.9 -> 32.8 mm
- net GND: track 105.3 -> 100.0 mm
- net Net-(J1-CC2): track 19.1 -> 21.1 mm

Commit message: Conmpleted design
Routing:
- net GND: track 100.0 -> 88.4 mm
- net Net-(J1-CC2): track 21.1 -> 22.5 mm
- net Net-(J1-CC1): track 11.8 -> 12.6 mm
Changed lines of the file:
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@@
 		(tags "resistor")
 		(property "Reference" "R2"
-			(at 1.5 0 360)
+			(at 1.5 0 0)
 			(layer "B.SilkS")
 			(effects
@@
 		)
 		(property "Value" "5.1k"
-			(at -1.5 0 360)
+			(at -1.5 0 0)
 			(layer "B.SilkS")
 			(effects
@@
 	)
 	(segment
-		(start 78.5 71.550352)
-		(end 77.65 70.700352)
+		(start 77.65 71.65)
+		(end 77.65 69.29)
 		(width 0.2)
 		(layer "F.Cu")
@@
 	)
 	(segment
-		(start 78.5 72.4)
-		(end 78.5 71.550352)
+		(start 77.38241 68.415)
+		(end 77.65 68.68259)
 		(width 0.2)
 		(layer "F.Cu")
@@
 	)
 	(segment
-		(start 77.65 70.700352)
+		(start 77.65 68.68259)
 		(end 77.65 69.29)
 		(width 0.2)
@@
 	)
 	(segment
-		(start 77.38241 68.415)
-		(end 77.65 68.68259)
+		(start 76.65 69.29)
+		(end 76.65 68.68259)
 		(width 0.2)
 		(layer "F.Cu")
@@
 	)
 	(segment
-		(start 77.65 68.68259)
-		(end 77.65 69.29)
+		(start 78.5 73.4)
+		(end 78.5 72.5)
 		(width 0.2)
 		(layer "F.Cu")
@@
 	)
 	(segment
-		(start 76.65 69.29)
-		(end 76.65 68.68259)
+		(start 78.5 72.5)
+		(end 77.65 71.65)
 		(width 0.2)
 		(layer "F.Cu")
@@
 	)
 	(via
-		(at 78.5 72.4)
+		(at 78.5 73.4)
 		(size 0.6)
 		(drill 0.3)
@@
 	)
 	(segment
-		(start 78.5 72.4)
-		(end 78.5 74.5)
+		(start 79.8825 75.8825)
+		(end 100.0125 75.8825)
 		(width 0.2)
 		(layer "B.Cu")
@@
 	)
 	(segment
-		(start 79.8825 75.8825)
-		(end 100.0125 75.8825)
+		(start 78.5 73.4)
+		(end 78.5 74.5)
 		(width 0.2)
 		(layer "B.Cu")
@@
 	)
 	(segment
-		(start 103.5 82.5)
-		(end 103.5 75)
+		(start 74 80)
+		(end 75.37 81.37)
 		(width 0.2)
 		(layer "B.Cu")
@@
 	)
 	(segment
-		(start 74 80)
-		(end 75.37 81.37)
+		(start 97.5 83.5)
+		(end 102 83.5)
 		(width 0.2)
 		(layer "B.Cu")
@@
 	)
 	(segment
-		(start 92 73.82)
-		(end 99.535 73.82)
+		(start 75.37 81.37)
+		(end 88.10625 81.37)
 		(width 0.2)
 		(layer "B.Cu")
@@
 	)
 	(segment
-		(start 75.37 81.37)
-		(end 88.10625 81.37)
+		(start 103 82.5)
+		(end 103 74.5)
 		(width 0.2)
 		(layer "B.Cu")
@@
 	)
 	(segment
-		(start 102.5 83.5)
-		(end 103.5 82.5)
+		(start 95.6575 73.3425)
+		(end 100.0125 73.3425)
 		(width 0.2)
 		(layer "B.Cu")
@@
 	)
 	(segment
-		(start 88 73.82)
-		(end 99.535 73.82)
+		(start 103 74.5)
+		(end 101.8425 73.3425)
 		(width 0.2)
 		(layer "B.Cu")
@@
 	)
 	(segment
-		(start 94.059375 81.37)
-		(end 94.689375 82)
+		(start 99.535 73.82)
+		(end 100.0125 73.3425)
 		(width 0.2)
 		(layer "B.Cu")
@@
 	)
 	(segment
-		(start 98 83.5)
-		(end 102.5 83.5)
+		(start 95.18 73.82)
+		(end 95.6575 73.3425)
 		(width 0.2)
 		(layer "B.Cu")
@@
 	)
 	(segment
-		(start 99.535 73.82)
-		(end 100.0125 73.3425)
+		(start 92 73.82)
+		(end 95.18 73.82)
 		(width 0.2)
 		(layer "B.Cu")
@@
 	)
 	(segment
-		(start 94.689375 82)
-		(end 96.5 82)
+		(start 95.37 81.37)
+		(end 97.5 83.5)
 		(width 0.2)
 		(layer "B.Cu")
@@
 	)
 	(segment
-		(start 96.5 82)
-		(end 98 83.5)
+		(start 102 83.5)
+		(end 103 82.5)
 		(width 0.2)
 		(layer "B.Cu")
@@
 	)
 	(segment
-		(start 103.5 75)
-		(end 101.8425 73.3425)
+		(start 94.059375 81.37)
+		(end 95.37 81.37)
 		(width 0.2)
 		(layer "B.Cu")
@@
 	)
 	(segment
-		(start 75.15 71.65)
+		(start 75.15 72.65)
 		(end 75.15 69.29)
 		(width 0.2)
@@
 	)
 	(segment
-		(start 79.5 73)
-		(end 76.5 73)
+		(start 76.5 74)
+		(end 75.15 72.65)
 		(width 0.2)
 		(layer "F.Cu")
@@
 	)
 	(segment
-		(start 76.5 73)
-		(end 75.15 71.65)
+		(start 79 74)
+		(end 76.5 74)
+		(width 0.2)
+		(layer "F.Cu")
+		(net 103)
+	)
+	(segment
+		(start 79.75 73.25)
+		(end 79 74)
 		(width 0.2)
 		(layer "F.Cu")
@@
 	)
 	(via
-		(at 79.5 73)
+		(at 79.75 73.25)
 		(size 0.6)
 		(drill 0.3)
@@
 	)
 	(segment
-		(start 81 71.5)
+		(start 81.5 71.5)
 		(end 90.32 71.5)
 		(width 0.2)
@@
 	)
 	(segment
-		(start 90.32 71.5)
-		(end 92 73.18)
+		(start 79.75 73.25)
+		(end 81.5 71.5)
 		(width 0.2)
 		(layer "B.Cu")
@@
 	)
 	(segment
-		(start 79.5 73)
-		(end 81 71.5)
+		(start 90.32 71.5)
+		(end 92 73.18)
 		(width 0.2)
 		(layer "B.Cu")
@@
 	(segment
 		(start 76.5 80)
-		(end 87.55125 80)
+		(end 77.055 80.555)
 		(width 0.2)
 		(layer "B.Cu")
@@
 	)
 	(segment
-		(start 94.8425 80.555)
-		(end 95.25 80.9625)
+		(start 77.055 80.555)
+		(end 88.10625 80.555)
 		(width 0.2)
 		(layer "B.Cu")
@@
 	)
 	(segment
-		(start 94.059375 80.555)
-		(end 94.8425 80.555)
+		(start 96.534375 80.9625)
+		(end 100.0125 80.9625)
 		(width 0.2)
 		(layer "B.Cu")
@@
 	)
 	(segment
-		(start 87.55125 80)
-		(end 88.10625 80.555)
+		(start 96.126875 80.555)
+		(end 96.534375 80.9625)
 		(width 0.2)
 		(layer "B.Cu")
@@
 	)
 	(segment
-		(start 95.25 80.9625)
-		(end 100.0125 80.9625)
+		(start 94.059375 80.555)
+		(end 96.126875 80.555)
 		(width 0.2)
 		(layer "B.Cu")
@@
 	)
 	(segment
-		(start 77.50056 72.00056)
-		(end 76.5 71)
+		(start 76.5 71.5)
+		(end 76.5 70.165)
 		(width 0.2)
 		(layer "F.Cu")
@@
 	)
 	(segment
-		(start 76.15 69.29)
-		(end 76.15 69.89741)
+		(start 77.50056 72.50056)
+		(end 76.5 71.5)
 		(width 0.2)
 		(layer "F.Cu")
@@
 	)
 	(segment
-		(start 76.15 69.89741)
-		(end 76.41759 70.165)
+		(start 76.15 69.29)
+		(end 76.15 69.89741)
 		(width 0.2)
 		(layer "F.Cu")
@@
 	)
 	(segment
-		(start 77.50056 72.4)
-		(end 77.50056 72.00056)
+		(start 76.15 69.89741)
+		(end 76.41759 70.165)
 		(width 0.2)
 		(layer "F.Cu")
@@
 	)
 	(segment
-		(start 76.5 71)
-		(end 76.5 70.165)
+		(start 77.15 69.89741)
+		(end 77.15 69.29)
 		(width 0.2)
 		(layer "F.Cu")
@@
 	)
 	(segment
-		(start 77.15 69.89741)
-		(end 77.15 69.29)
+		(start 76.88241 70.165)
+		(end 77.15 69.89741)
 		(width 0.2)
 		(layer "F.Cu")
@@
 	)
 	(segment
-		(start 76.88241 70.165)
-		(end 77.15 69.89741)
+		(start 77.50056 73.4)
+		(end 77.50056 72.50056)
 		(width 0.2)
 		(layer "F.Cu")
@@
 	)
 	(via
-		(at 77.50056 72.4)
+		(at 77.50056 73.4)
 		(size 0.6)
 		(drill 0.3)
@@
 	)
 	(segment
-		(start 77.50056 72.4)
+		(start 77.50056 73.4)
 		(end 77.50056 77.00056)
 		(width 0.2)
@@
 	)
 	(segment
-		(start 77.50056 77.00056)
-		(end 78.9225 78.4225)
+		(start 78.9225 78.4225)
+		(end 100.0125 78.4225)
 		(width 0.2)
 		(layer "B.Cu")
@@
 	)
 	(segment
-		(start 78.9225 78.4225)
-		(end 100.0125 78.4225)
+		(start 77.50056 77.00056)
+		(end 78.9225 78.4225)
 		(width 0.2)
 		(layer "B.Cu")
@@
 	)
 	(segment
-		(start 78.15 69.89741)
-		(end 78.15 69.29)
+		(start 79.5 72.5)
+		(end 78.15 71.15)
 		(width 0.2)
 		(layer "F.Cu")
@@
 	)
 	(segment
-		(start 80.75259 72.5)
-		(end 78.15 69.89741)
+		(start 85 72.5)
+		(end 79.5 72.5)
 		(width 0.2)
 		(layer "F.Cu")
@@
 	)
 	(segment
-		(start 85 72.5)
-		(end 80.75259 72.5)
+		(start 78.15 71.15)
+		(end 78.15 69.29)
 		(width 0.2)
 		(layer "F.Cu")
