File: PCB/PicoKeyboard/key_matrix.kicad_sch (KiCad schematic)
At the start: 170 parts

Commit message: Changed
Parts:
- D1, D10, D11, D12, D13, D14, D15, D16, D17, D18, D19, D2, D20, D21, D22, D23, D24, D25, D26, D27, D28, D29, D3, D30, D31, D32, D33, D34, D35, D36, D37, D38, D39, D4, D40, D41, D42, D43, D44, D45, D46, D47, D48, D49, D5, D50, D51, D52, D53, D54, D55, D56, D57, D58, D59, D6, D60, D61, D62, D63, D64, D65, D66, D67, D68, D69, D7, D70, D71, D72, D73, D74, D75, D76, D77, D78, D79, D8, D80, D81, D82, D83, D84, D85, D9: footprint (none) -> ScottoKeebs_Components:Diode_SOD-123
- S1, S10, S11, S12, S13, S14, S15, S16, S17, S18, S19, S2, S20, S21, S22, S23, S24, S25, S26, S27, S29, S3, S30, S31, S33, S34, S35, S36, S37, S38, S39, S4, S40, S41, S42, S43, S44, S46, S47, S48, S5, S50, S51, S52, S53, S54, S55, S56, S57, S58, S59, S6, S60, S63, S64, S65, S66, S67, S68, S69, S7, S70, S71, S72, S74, S8, S83, S84, S85, S9: footprint (none) -> Button_Switch_Keyboard:SW_Cherry_MX_1.00u_PCB
- S28: footprint (none) -> Button_Switch_Keyboard:SW_Cherry_MX_2.00u_PCB
- S32, S45: footprint (none) -> Button_Switch_Keyboard:SW_Cherry_MX_1.50u_PCB
- S49: footprint (none) -> Button_Switch_Keyboard:SW_Cherry_MX_1.75u_PCB
- S61, S62: footprint (none) -> Button_Switch_Keyboard:SW_Cherry_MX_2.25u_PCB
- S73: footprint (none) -> Button_Switch_Keyboard:SW_Cherry_MX_2.75u_PCB
- S75, S76, S77, S79, S80, S81, S82: footprint (none) -> Button_Switch_Keyboard:SW_Cherry_MX_1.25u_PCB
- S78: footprint (none) -> Button_Switch_Keyboard:SW_Cherry_MX_6.25u_PCB
Connections:
- net C1: now also S15.1, S62.1; no longer S14.1, S61.1
- net C10: now also S24.1; no longer S23.1
- net C11: now also S25.1; no longer S24.1
- net C12: now also S26.1; no longer S25.1
- net C13: now also S27.1; no longer S26.1
- net C14: now also S14.1, S61.1; no longer S27.1, S62.1
- net C2: now also S16.1; no longer S15.1
- net C3: now also S17.1; no longer S16.1
- net C4: now also S18.1; no longer S17.1
- net C5: now also S19.1; no longer S18.1
- net C6: now also S20.1; no longer S19.1
- net C7: now also S21.1; no longer S20.1
- net C8: now also S22.1; no longer S21.1
- net C9: now also S23.1; no longer S22.1
- net R1: now also D14.1 (K); no longer D27.1 (K)
- net R2: now also D27.1 (K); no longer D14.1 (K)
- net R4: now also D61.1 (K); no longer D62.1 (K)
- net R5: now also D62.1 (K); no longer D61.1 (K)
Other:
- moved on the sheet: D14, D15, D16, D17, D18, D19, D20, D21, D22, D23, D24, D25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

Commit message: Update PCB
Parts:
- S1: value Keyswitch -> Esc
- S10: value Keyswitch -> F9
- S11: value Keyswitch -> F10
- S12: value Keyswitch -> F11
- S13: value Keyswitch -> F12
- S14: value Keyswitch -> Print
- S15: value Keyswitch -> Ins
- S16: value Keyswitch -> Del
- S17: value Keyswitch -> Tilde
- S18: value Keyswitch -> 1
- S19: value Keyswitch -> 2
- S2: value Keyswitch -> F1
- S20: value Keyswitch -> 3
- S21: value Keyswitch -> 4
- S22: value Keyswitch -> 5
- S23: value Keyswitch -> 6
- S24: value Keyswitch -> 7
- S25: value Keyswitch -> 8
- S26: value Keyswitch -> 9
- S27: value Keyswitch -> 0
- S28: value Keyswitch -> -; footprint Button_Switch_Keyboard:SW_Cherry_MX_2.00u_PCB -> Button_Switch_Keyboard:SW_Cherry_MX_1.00u_PCB
- S29: value Keyswitch -> =
- S3: value Keyswitch -> F2
- S30: value Keyswitch -> Backspace; footprint Button_Switch_Keyboard:SW_Cherry_MX_1.00u_PCB -> Button_Switch_Keyboard:SW_Cherry_MX_2.00u_PCB
- S31: value Keyswitch -> Home
- S32: value Keyswitch -> End; footprint Button_Switch_Keyboard:SW_Cherry_MX_1.50u_PCB -> Button_Switch_Keyboard:SW_Cherry_MX_1.00u_PCB
- S33: value Keyswitch -> Tab; footprint Button_Switch_Keyboard:SW_Cherry_MX_1.00u_PCB -> Button_Switch_Keyboard:SW_Cherry_MX_1.50u_PCB
- S34: value Keyswitch -> Q
- S35: value Keyswitch -> W
- S36: value Keyswitch -> E
- S37: value Keyswitch -> R
- S38: value Keyswitch -> T
- S39: value Keyswitch -> Y
- S4: value Keyswitch -> F3
- S40: value Keyswitch -> U
- S41: value Keyswitch -> I
- S42: value Keyswitch -> O
- S43: value Keyswitch -> P
- S44: value Keyswitch -> [
- S45: value Keyswitch -> ]; footprint Button_Switch_Keyboard:SW_Cherry_MX_1.50u_PCB -> Button_Switch_Keyboard:SW_Cherry_MX_1.00u_PCB
- S46: value Keyswitch -> \|; footprint Button_Switch_Keyboard:SW_Cherry_MX_1.00u_PCB -> Button_Switch_Keyboard:SW_Cherry_MX_1.50u_PCB
- S47: value Keyswitch -> PgDn
- S48: value Keyswitch -> CapsLock; footprint Button_Switch_Keyboard:SW_Cherry_MX_1.00u_PCB -> Button_Switch_Keyboard:SW_Cherry_MX_1.75u_PCB
- S49: value Keyswitch -> A; footprint Button_Switch_Keyboard:SW_Cherry_MX_1.75u_PCB -> Button_Switch_Keyboard:SW_Cherry_MX_1.00u_PCB
- S5: value Keyswitch -> F4
- S50: value Keyswitch -> S
- S51: value Keyswitch -> D
- S52: value Keyswitch -> F
- S53: value Keyswitch -> G
- S54: value Keyswitch -> H
- S55: value Keyswitch -> J
- S56: value Keyswitch -> K
- S57: value Keyswitch -> L
- S58: value Keyswitch -> ;:
- S59: value Keyswitch -> '"
- S6: value Keyswitch -> F5
- S60: value Keyswitch -> Enter; footprint Button_Switch_Keyboard:SW_Cherry_MX_1.00u_PCB -> Button_Switch_Keyboard:SW_Cherry_MX_2.25u_PCB
- S61: value Keyswitch -> PgUp; footprint Button_Switch_Keyboard:SW_Cherry_MX_2.25u_PCB -> Button_Switch_Keyboard:SW_Cherry_MX_1.00u_PCB
- S62: value Keyswitch -> L.Shift
- S63: value Keyswitch -> Z
- S64: value Keyswitch -> X
- S65: value Keyswitch -> C
- S66: value Keyswitch -> V
- S67: value Keyswitch -> B
- S68: value Keyswitch -> N
- S69: value Keyswitch -> M
- S7: value Keyswitch -> F6
- S70: value Keyswitch -> ,<
- S71: value Keyswitch -> .>
- S72: value Keyswitch -> /?
- S73: value Keyswitch -> R.Shift
- S74, S85: value Keyswitch -> Up
- S75: value Keyswitch -> L.Ctrl
- S76: value Keyswitch -> L.Super
- S77: value Keyswitch -> L.Alt
- S78: value Keyswitch -> Space
- S79: value Keyswitch -> Fn; footprint Button_Switch_Keyboard:SW_Cherry_MX_1.25u_PCB -> Button_Switch_Keyboard:SW_Cherry_MX_1.00u_PCB
- S8: value Keyswitch -> F7
- S80: value Keyswitch -> Custom 1; footprint Button_Switch_Keyboard:SW_Cherry_MX_1.25u_PCB -> Button_Switch_Keyboard:SW_Cherry_MX_1.00u_PCB
- S81: value Keyswitch -> Custom 2; footprint Button_Switch_Keyboard:SW_Cherry_MX_1.25u_PCB -> Button_Switch_Keyboard:SW_Cherry_MX_1.00u_PCB
- S82: value Keyswitch -> Custom 3; footprint Button_Switch_Keyboard:SW_Cherry_MX_1.25u_PCB -> Button_Switch_Keyboard:SW_Cherry_MX_1.00u_PCB
- S83: value Keyswitch -> Left
- S84: value Keyswitch -> Down
- S9: value Keyswitch -> F8
Connections:
- net C1: now also S17.1, S33.1, S48.1; no longer S15.1, S32.1, S49.1
- net C10: now also S26.1, S42.1, S57.1; no longer S24.1, S41.1, S58.1
- net C11: now also S27.1, S43.1, S58.1; no longer S25.1, S42.1, S59.1
- net C12: now also S28.1, S44.1, S59.1; no longer S26.1, S43.1, S60.1
- net C13: now also S29.1, S45.1; no longer S27.1, S44.1
- net C14: now also S30.1, S46.1, S60.1, S83.1; no longer S28.1, S45.1, S61.1
- net C15: now also S15.1, S31.1, S47.1, S61.1, S74.1, S84.1; no longer S29.1, S46.1, S83.1
- net C16: now also S16.1, S32.1, S85.1; no longer S30.1, S47.1, S74.1, S84.1
- net C2: now also S18.1, S34.1, S49.1; no longer S16.1, S33.1, S50.1
- net C3: now also S19.1, S35.1, S50.1; no longer S17.1, S34.1, S51.1
- net C4: now also S20.1, S36.1, S51.1; no longer S18.1, S35.1, S52.1
- net C5: now also S21.1, S37.1, S52.1; no longer S19.1, S36.1, S53.1
- net C6: now also S22.1, S38.1, S53.1; no longer S20.1, S37.1, S54.1
- net C7: now also S23.1, S39.1, S54.1; no longer S21.1, S38.1, S55.1
- net C8: now also S24.1, S40.1, S55.1; no longer S22.1, S39.1, S56.1
- net C9: now also S25.1, S41.1, S56.1; no longer S23.1, S40.1, S57.1
- net R1: now also D15.1 (K), D16.1 (K)
- net R2: now also D32.1 (K); no longer D15.1 (K), D16.1 (K)
- net R3: no longer D32.1 (K), D48.1 (K)
- net R4: now also D48.1 (K)
- removed net C17: S31.1, S48.1, S85.1
Other:
- moved on the sheet: D17, D18, D19, D20, D21, D22, D23, D24, D25, D26, D27, D28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

Commit message: New layout
Parts:
- removed D77, D78, D79, D80, D81, D82, D83, D84, D85: Diode, ScottoKeebs_Components:Diode_SOD-123, symbol ScottoKeebs:Placeholder_Diode
- removed S77: L.Alt, Button_Switch_Keyboard:SW_Cherry_MX_1.25u_PCB, symbol ScottoKeebs:Placeholder_Keyswitch
- removed S78: Space, Button_Switch_Keyboard:SW_Cherry_MX_6.25u_PCB, symbol ScottoKeebs:Placeholder_Keyswitch
- removed S79: Fn, Button_Switch_Keyboard:SW_Cherry_MX_1.00u_PCB, symbol ScottoKeebs:Placeholder_Keyswitch
- removed S80: Custom 1, Button_Switch_Keyboard:SW_Cherry_MX_1.00u_PCB, symbol ScottoKeebs:Placeholder_Keyswitch
- removed S81: Custom 2, Button_Switch_Keyboard:SW_Cherry_MX_1.00u_PCB, symbol ScottoKeebs:Placeholder_Keyswitch
- removed S82: Custom 3, Button_Switch_Keyboard:SW_Cherry_MX_1.00u_PCB, symbol ScottoKeebs:Placeholder_Keyswitch
- removed S83: Left, Button_Switch_Keyboard:SW_Cherry_MX_1.00u_PCB, symbol ScottoKeebs:Placeholder_Keyswitch
- removed S84: Down, Button_Switch_Keyboard:SW_Cherry_MX_1.00u_PCB, symbol ScottoKeebs:Placeholder_Keyswitch
- removed S85: Up, Button_Switch_Keyboard:SW_Cherry_MX_1.00u_PCB, symbol ScottoKeebs:Placeholder_Keyswitch
- S1, S10, S11, S12, S13, S2, S3, S4, S5, S6, S7, S8, S9: footprint Button_Switch_Keyboard:SW_Cherry_MX_1.00u_PCB -> ScottoKeebs_MX:MX_PCB_1.00u
- S14: value Print -> Del; footprint Button_Switch_Keyboard:SW_Cherry_MX_1.00u_PCB -> ScottoKeebs_MX:MX_PCB_1.00u
- S15: value Ins -> Backtick; footprint Button_Switch_Keyboard:SW_Cherry_MX_1.00u_PCB -> ScottoKeebs_MX:MX_PCB_1.00u
- S16: value Del -> Num_1; footprint Button_Switch_Keyboard:SW_Cherry_MX_1.00u_PCB -> ScottoKeebs_MX:MX_PCB_1.00u
- S17: value Tilde -> Num_2; footprint Button_Switch_Keyboard:SW_Cherry_MX_1.00u_PCB -> ScottoKeebs_MX:MX_PCB_1.00u
- S18: value 1 -> Num_3; footprint Button_Switch_Keyboard:SW_Cherry_MX_1.00u_PCB -> ScottoKeebs_MX:MX_PCB_1.00u
- S19: value 2 -> Num_4; footprint Button_Switch_Keyboard:SW_Cherry_MX_1.00u_PCB -> ScottoKeebs_MX:MX_PCB_1.00u
- S20: value 3 -> Num_5; footprint Button_Switch_Keyboard:SW_Cherry_MX_1.00u_PCB -> ScottoKeebs_MX:MX_PCB_1.00u
- S21: value 4 -> Num_6; footprint Button_Switch_Keyboard:SW_Cherry_MX_1.00u_PCB -> ScottoKeebs_MX:MX_PCB_1.00u
- S22: value 5 -> Num_7; footprint Button_Switch_Keyboard:SW_Cherry_MX_1.00u_PCB -> ScottoKeebs_MX:MX_PCB_1.00u
- S23: value 6 -> Num_8; footprint Button_Switch_Keyboard:SW_Cherry_MX_1.00u_PCB -> ScottoKeebs_MX:MX_PCB_1.00u
- S24: value 7 -> Num_9; footprint Button_Switch_Keyboard:SW_Cherry_MX_1.00u_PCB -> ScottoKeebs_MX:MX_PCB_1.00u
- S25: value 8 -> Num_0; footprint Button_Switch_Keyboard:SW_Cherry_MX_1.00u_PCB -> ScottoKeebs_MX:MX_PCB_1.00u
- S26: value 9 -> Minus; footprint Button_Switch_Keyboard:SW_Cherry_MX_1.00u_PCB -> ScottoKeebs_MX:MX_PCB_1.00u
- S27: value 0 -> Add; footprint Button_Switch_Keyboard:SW_Cherry_MX_1.00u_PCB -> ScottoKeebs_MX:MX_PCB_1.00u
- S28: value - -> Backspace; footprint Button_Switch_Keyboard:SW_Cherry_MX_1.00u_PCB -> ScottoKeebs_MX:MX_PCB_2.00u
- S29: value = -> Tab; footprint Button_Switch_Keyboard:SW_Cherry_MX_1.00u_PCB -> ScottoKeebs_MX:MX_PCB_1.50u
- S30: value Backspace -> Q; footprint Button_Switch_Keyboard:SW_Cherry_MX_2.00u_PCB -> ScottoKeebs_MX:MX_PCB_1.00u
- S31: value Home -> W; footprint Button_Switch_Keyboard:SW_Cherry_MX_1.00u_PCB -> ScottoKeebs_MX:MX_PCB_1.00u
- S32: value End -> E; footprint Button_Switch_Keyboard:SW_Cherry_MX_1.00u_PCB -> ScottoKeebs_MX:MX_PCB_1.00u
- S33: value Tab -> R; footprint Button_Switch_Keyboard:SW_Cherry_MX_1.50u_PCB -> ScottoKeebs_MX:MX_PCB_1.00u
- S34: value Q -> T; footprint Button_Switch_Keyboard:SW_Cherry_MX_1.00u_PCB -> ScottoKeebs_MX:MX_PCB_1.00u
- S35: value W -> Y; footprint Button_Switch_Keyboard:SW_Cherry_MX_1.00u_PCB -> ScottoKeebs_MX:MX_PCB_1.00u
- S36: value E -> U; footprint Button_Switch_Keyboard:SW_Cherry_MX_1.00u_PCB -> ScottoKeebs_MX:MX_PCB_1.00u
- S37: value R -> I; footprint Button_Switch_Keyboard:SW_Cherry_MX_1.00u_PCB -> ScottoKeebs_MX:MX_PCB_1.00u
- S38: value T -> O; footprint Button_Switch_Keyboard:SW_Cherry_MX_1.00u_PCB -> ScottoKeebs_MX:MX_PCB_1.00u
- S39: value Y -> P; footprint Button_Switch_Keyboard:SW_Cherry_MX_1.00u_PCB -> ScottoKeebs_MX:MX_PCB_1.00u
- S40: value U -> [; footprint Button_Switch_Keyboard:SW_Cherry_MX_1.00u_PCB -> ScottoKeebs_MX:MX_PCB_1.00u
- S41: value I -> ]; footprint Button_Switch_Keyboard:SW_Cherry_MX_1.00u_PCB -> ScottoKeebs_MX:MX_PCB_1.00u
- S42: value O -> Pipe; footprint Button_Switch_Keyboard:SW_Cherry_MX_1.00u_PCB -> ScottoKeebs_MX:MX_PCB_1.50u
- S43: value P -> Caps; footprint Button_Switch_Keyboard:SW_Cherry_MX_1.00u_PCB -> ScottoKeebs_MX:MX_PCB_1.75u
- S44: value [ -> A; footprint Button_Switch_Keyboard:SW_Cherry_MX_1.00u_PCB -> ScottoKeebs_MX:MX_PCB_1.00u
- S45: value ] -> S; footprint Button_Switch_Keyboard:SW_Cherry_MX_1.00u_PCB -> ScottoKeebs_MX:MX_PCB_1.00u
- S46: value \| -> D; footprint Button_Switch_Keyboard:SW_Cherry_MX_1.50u_PCB -> ScottoKeebs_MX:MX_PCB_1.00u
- S47: value PgDn -> F; footprint Button_Switch_Keyboard:SW_Cherry_MX_1.00u_PCB -> ScottoKeebs_MX:MX_PCB_1.00u
- S48: value CapsLock -> G; footprint Button_Switch_Keyboard:SW_Cherry_MX_1.75u_PCB -> ScottoKeebs_MX:MX_PCB_1.00u
- S49: value A -> H; footprint Button_Switch_Keyboard:SW_Cherry_MX_1.00u_PCB -> ScottoKeebs_MX:MX_PCB_1.00u
- S50: value S -> J; footprint Button_Switch_Keyboard:SW_Cherry_MX_1.00u_PCB -> ScottoKeebs_MX:MX_PCB_1.00u
- S51: value D -> K; footprint Button_Switch_Keyboard:SW_Cherry_MX_1.00u_PCB -> ScottoKeebs_MX:MX_PCB_1.00u
- S52: value F -> L; footprint Button_Switch_Keyboard:SW_Cherry_MX_1.00u_PCB -> ScottoKeebs_MX:MX_PCB_1.00u
- S53: value G -> Semicolon; footprint Button_Switch_Keyboard:SW_Cherry_MX_1.00u_PCB -> ScottoKeebs_MX:MX_PCB_1.00u
- S54: value H -> Quote; footprint Button_Switch_Keyboard:SW_Cherry_MX_1.00u_PCB -> ScottoKeebs_MX:MX_PCB_1.00u
- S55: value J -> Enter; footprint Button_Switch_Keyboard:SW_Cherry_MX_1.00u_PCB -> ScottoKeebs_MX:MX_PCB_2.25u
- S56: value K -> L.Shift; footprint Button_Switch_Keyboard:SW_Cherry_MX_1.00u_PCB -> ScottoKeebs_MX:MX_PCB_2.25u
- S57: value L -> Z; footprint Button_Switch_Keyboard:SW_Cherry_MX_1.00u_PCB -> ScottoKeebs_MX:MX_PCB_1.00u
- S58: value ;: -> X; footprint Button_Switch_Keyboard:SW_Cherry_MX_1.00u_PCB -> ScottoKeebs_MX:MX_PCB_1.00u
- S59: value '" -> C; footprint Button_Switch_Keyboard:SW_Cherry_MX_1.00u_PCB -> ScottoKeebs_MX:MX_PCB_1.00u
- S60: value Enter -> V; footprint Button_Switch_Keyboard:SW_Cherry_MX_2.25u_PCB -> ScottoKeebs_MX:MX_PCB_1.00u
- S61: value PgUp -> B; footprint Button_Switch_Keyboard:SW_Cherry_MX_1.00u_PCB -> ScottoKeebs_MX:MX_PCB_1.00u
- S62: value L.Shift -> N; footprint Button_Switch_Keyboard:SW_Cherry_MX_2.25u_PCB -> ScottoKeebs_MX:MX_PCB_1.00u
- S63: value Z -> M; footprint Button_Switch_Keyboard:SW_Cherry_MX_1.00u_PCB -> ScottoKeebs_MX:MX_PCB_1.00u
- S64: value X -> Comma; footprint Button_Switch_Keyboard:SW_Cherry_MX_1.00u_PCB -> ScottoKeebs_MX:MX_PCB_1.00u
- S65: value C -> Period; footprint Button_Switch_Keyboard:SW_Cherry_MX_1.00u_PCB -> ScottoKeebs_MX:MX_PCB_1.00u
- S66: value V -> Slash; footprint Button_Switch_Keyboard:SW_Cherry_MX_1.00u_PCB -> ScottoKeebs_MX:MX_PCB_1.00u
- S67: value B -> R.Shift; footprint Button_Switch_Keyboard:SW_Cherry_MX_1.00u_PCB -> ScottoKeebs_MX:MX_PCB_2.75u
- S68: value N -> Ctrl; footprint Button_Switch_Keyboard:SW_Cherry_MX_1.00u_PCB -> ScottoKeebs_MX:MX_PCB_1.25u
- S69: value M -> Super; footprint Button_Switch_Keyboard:SW_Cherry_MX_1.00u_PCB -> ScottoKeebs_MX:MX_PCB_1.25u
- S70: value ,< -> Alt; footprint Button_Switch_Keyboard:SW_Cherry_MX_1.00u_PCB -> ScottoKeebs_MX:MX_PCB_1.25u
- S71: value .> -> Space; footprint Button_Switch_Keyboard:SW_Cherry_MX_1.00u_PCB -> ScottoKeebs_MX:MX_PCB_6.25u
- S72: value /? -> Fn; footprint Button_Switch_Keyboard:SW_Cherry_MX_1.00u_PCB -> ScottoKeebs_MX:MX_PCB_1.00u
- S73: value R.Shift -> Custom_1; footprint Button_Switch_Keyboard:SW_Cherry_MX_2.75u_PCB -> ScottoKeebs_MX:MX_PCB_1.00u
- S74: value Up -> Custom_2; footprint Button_Switch_Keyboard:SW_Cherry_MX_1.00u_PCB -> ScottoKeebs_MX:MX_PCB_1.00u
- S75: value L.Ctrl -> Custom_3; footprint Button_Switch_Keyboard:SW_Cherry_MX_1.25u_PCB -> ScottoKeebs_MX:MX_PCB_1.00u
- S76: value L.Super -> Custom_4; footprint Button_Switch_Keyboard:SW_Cherry_MX_1.25u_PCB -> ScottoKeebs_MX:MX_PCB_1.00u
Connections:
- net R6 is gone; now on net R5: D75.1 (K), D76.1 (K)
- net C1: now also S16.1, S2.1, S30.1, S44.1, S57.1, S69.1; no longer S1.1, S17.1, S33.1, S48.1, S62.1, S75.1
- net C10: now also S11.1, S25.1, S39.1, S53.1, S66.1, S67.1; no longer S10.1, S26.1, S42.1, S57.1, S71.1
- net C11: now also S12.1, S26.1, S28.1, S40.1, S54.1; no longer S11.1, S27.1, S43.1, S58.1, S72.1
- net C12: now also S13.1, S14.1, S27.1, S41.1, S42.1; no longer S12.1, S28.1, S44.1, S59.1
- net C2: now also S17.1, S3.1, S31.1, S45.1, S58.1, S70.1; no longer S18.1, S2.1, S34.1, S49.1, S63.1, S76.1
- net C3: now also S18.1, S32.1, S4.1, S46.1, S59.1, S71.1; no longer S19.1, S3.1, S35.1, S50.1, S64.1
- net C4: now also S19.1, S33.1, S47.1, S5.1, S60.1, S72.1; no longer S20.1, S36.1, S4.1, S51.1, S65.1
- net C5: now also S20.1, S34.1, S48.1, S6.1, S61.1, S73.1; no longer S21.1, S37.1, S5.1, S52.1, S66.1
- net C6: now also S21.1, S35.1, S49.1, S62.1, S7.1, S74.1; no longer S22.1, S38.1, S53.1, S6.1, S67.1
- net C7: now also S22.1, S36.1, S50.1, S63.1, S75.1, S8.1; no longer S23.1, S39.1, S54.1, S68.1, S7.1
- net C8: now also S23.1, S37.1, S51.1, S64.1, S76.1, S9.1; no longer S24.1, S40.1, S55.1, S69.1, S8.1
- net C9: now also S10.1, S24.1, S38.1, S52.1, S55.1, S65.1; no longer S25.1, S41.1, S56.1, S70.1, S9.1
- net R1: now also D17.1 (K), D18.1 (K), D19.1 (K), D20.1 (K), D21.1 (K), D22.1 (K), D23.1 (K), D24.1 (K), D25.1 (K), D26.1 (K), D27.1 (K); no longer D1.1 (K), D10.1 (K), D11.1 (K), D12.1 (K), D13.1 (K), D14.1 (K), D2.1 (K), D3.1 (K), D4.1 (K), D5.1 (K), D6.1 (K), D7.1 (K), D8.1 (K), D9.1 (K)
- net R2: now also D33.1 (K), D34.1 (K), D35.1 (K), D36.1 (K), D37.1 (K), D38.1 (K), D39.1 (K), D40.1 (K), D41.1 (K); no longer D17.1 (K), D18.1 (K), D19.1 (K), D20.1 (K), D21.1 (K), D22.1 (K), D23.1 (K), D24.1 (K), D25.1 (K), D26.1 (K), D27.1 (K), D28.1 (K)
- net R3: now also D14.1 (K), D48.1 (K), D49.1 (K), D50.1 (K), D51.1 (K), D52.1 (K), D53.1 (K), D54.1 (K); no longer D33.1 (K), D34.1 (K), D35.1 (K), D36.1 (K), D37.1 (K), D38.1 (K), D39.1 (K), D40.1 (K), D41.1 (K), D42.1 (K)
- net R4: now also D28.1 (K), D42.1 (K), D62.1 (K), D63.1 (K), D64.1 (K), D65.1 (K), D66.1 (K); no longer D48.1 (K), D49.1 (K), D50.1 (K), D51.1 (K), D52.1 (K), D53.1 (K), D54.1 (K), D55.1 (K)
- net R5: now also D55.1 (K); no longer D62.1 (K), D63.1 (K), D64.1 (K), D65.1 (K), D66.1 (K)
- removed net C13: S13.1, S29.1, S45.1
- removed net C14: S14.1, S30.1, S46.1, S60.1, S73.1
- removed net C15: S15.1, S31.1, S47.1, S61.1, S74.1
- removed net C16: S16.1, S32.1
- new net C0: S1.1, S15.1, S29.1, S43.1, S56.1, S68.1
- new net R0: D1.1 (K), D10.1 (K), D11.1 (K), D12.1 (K), D13.1 (K), D2.1 (K), D3.1 (K), D4.1 (K), D5.1 (K), D6.1 (K), D7.1 (K), D8.1 (K), D9.1 (K)

Commit message: Change layout
Parts:
- added D77: Diode, ScottoKeebs_Components:Diode_SOD-123, symbol ScottoKeebs:Placeholder_Diode
- added S77: Del, ScottoKeebs_MX:MX_Plate_1.00u, symbol ScottoKeebs:Placeholder_Keyswitch
- S1, S10, S11, S12, S13, S15, S16, S17, S18, S19, S2, S20, S21, S22, S23, S24, S25, S26, S27, S3, S30, S31, S32, S33, S34, S35, S36, S37, S38, S39, S4, S40, S41, S44, S45, S46, S47, S48, S49, S5, S50, S51, S52, S53, S54, S57, S58, S59, S6, S60, S61, S62, S63, S64, S65, S66, S7, S73, S74, S75, S76, S8, S9: footprint ScottoKeebs_MX:MX_PCB_1.00u -> ScottoKeebs_MX:MX_Plate_1.00u
- S14: value Del -> Print; footprint ScottoKeebs_MX:MX_PCB_1.00u -> ScottoKeebs_MX:MX_Plate_1.00u
- S28: footprint ScottoKeebs_MX:MX_PCB_2.00u -> ScottoKeebs_MX:MX_Plate_2.00u
- S29, S42: footprint ScottoKeebs_MX:MX_PCB_1.50u -> ScottoKeebs_MX:MX_Plate_1.50u
- S43: footprint ScottoKeebs_MX:MX_PCB_1.75u -> ScottoKeebs_MX:MX_Plate_1.75u
- S55, S56: footprint ScottoKeebs_MX:MX_PCB_2.25u -> ScottoKeebs_MX:MX_Plate_2.25u
- S67: footprint ScottoKeebs_MX:MX_PCB_2.75u -> ScottoKeebs_MX:MX_Plate_2.75u
- S68, S69, S70: footprint ScottoKeebs_MX:MX_PCB_1.25u -> ScottoKeebs_MX:MX_Plate_1.25u
- S71: value Space -> Fn; footprint ScottoKeebs_MX:MX_PCB_6.25u -> ScottoKeebs_MX:MX_Plate_1.00u
- S72: value Fn -> Space; footprint ScottoKeebs_MX:MX_PCB_1.00u -> ScottoKeebs_MX:MX_Plate_6.25u
Connections:
- net C10: now also S77.1; no longer S67.1
- net C11: now also S67.1
- net C12: now also S55.1; no longer S14.1
- net C9: now also S14.1; no longer S55.1
- net R3: now also D42.1 (K); no longer D14.1 (K)
- net R4: now also D55.1 (K), D67.1 (K); no longer D28.1 (K), D42.1 (K)
- net R5: now also D14.1 (K), D28.1 (K), D77.1 (K); no longer D55.1 (K), D67.1 (K)
- new net: D77.2 (A), S77.2
Other:
- moved on the sheet: D14, D28, D42, D55, D67, S14, S28, S42, S55, S67

Commit message: Fix
Parts:
- S1, S10, S11, S12, S13, S14, S15, S16, S17, S18, S19, S2, S20, S21, S22, S23, S24, S25, S26, S27, S3, S30, S31, S32, S33, S34, S35, S36, S37, S38, S39, S4, S40, S41, S44, S45, S46, S47, S48, S49, S5, S50, S51, S52, S53, S54, S57, S58, S59, S6, S60, S61, S62, S63, S64, S65, S66, S7, S71, S73, S74, S75, S76, S77, S8, S9: footprint ScottoKeebs_MX:MX_Plate_1.00u -> ScottoKeebs_MX:MX_PCB_1.00u
- S28: footprint ScottoKeebs_MX:MX_Plate_2.00u -> ScottoKeebs_MX:MX_PCB_2.00u
- S29, S42: footprint ScottoKeebs_MX:MX_Plate_1.50u -> ScottoKeebs_MX:MX_PCB_1.50u
- S43: footprint ScottoKeebs_MX:MX_Plate_1.75u -> ScottoKeebs_MX:MX_PCB_1.75u
- S55, S56: footprint ScottoKeebs_MX:MX_Plate_2.25u -> ScottoKeebs_MX:MX_PCB_2.25u
- S67: footprint ScottoKeebs_MX:MX_Plate_2.75u -> ScottoKeebs_MX:MX_PCB_2.75u
- S68, S69, S70: footprint ScottoKeebs_MX:MX_Plate_1.25u -> ScottoKeebs_MX:MX_PCB_1.25u
- S72: footprint ScottoKeebs_MX:MX_Plate_6.25u -> ScottoKeebs_MX:MX_PCB_6.25u

Commit message: Hotswap
Parts:
- S1, S10, S11, S12, S13, S14, S15, S16, S17, S18, S19, S2, S20, S21, S22, S23, S24, S25, S26, S27, S3, S30, S31, S32, S33, S34, S35, S36, S37, S38, S39, S4, S40, S41, S44, S45, S46, S47, S48, S49, S5, S50, S51, S52, S53, S54, S57, S58, S59, S6, S60, S61, S62, S63, S64, S65, S66, S7, S71, S73, S74, S75, S76, S77, S8, S9: footprint ScottoKeebs_MX:MX_PCB_1.00u -> ScottoKeebs_Hotswap:Hotswap_MX_1.00u
- S28: footprint ScottoKeebs_MX:MX_PCB_2.00u -> ScottoKeebs_Hotswap:Hotswap_MX_2.00u
- S29, S42: footprint ScottoKeebs_MX:MX_PCB_1.50u -> ScottoKeebs_Hotswap:Hotswap_MX_1.50u
- S43: footprint ScottoKeebs_MX:MX_PCB_1.75u -> ScottoKeebs_Hotswap:Hotswap_MX_1.75u
- S55, S56: footprint ScottoKeebs_MX:MX_PCB_2.25u -> ScottoKeebs_Hotswap:Hotswap_MX_2.25u
- S67: footprint ScottoKeebs_MX:MX_PCB_2.75u -> ScottoKeebs_Hotswap:Hotswap_MX_2.75u
- S68, S69, S70: footprint ScottoKeebs_MX:MX_PCB_1.25u -> ScottoKeebs_Hotswap:Hotswap_MX_1.25u
- S72: footprint ScottoKeebs_MX:MX_PCB_6.25u -> ScottoKeebs_Hotswap:Hotswap_MX_6.25u
Connections:
- net C10: now also S28.1; no longer S77.1
- net C11: now also S77.1; no longer S28.1
- net C12: now also S14.1; no longer S42.1
- net C9: now also S42.1; no longer S14.1
- net R3: now also D55.1 (K); no longer D42.1 (K)
- net R4: no longer D55.1 (K)
- net R5: now also D42.1 (K)
Other:
- moved on the sheet: D14, D28, D42, D55, D77, S14, S28, S42, S55, S77

Commit message: Update PCB
Connections:
- net C10: now also S55.1; no longer S28.1
- net C11: now also S14.1, S42.1; no longer S67.1, S77.1
- net C12: now also S28.1, S77.1; no longer S14.1, S55.1
- net C9: now also S67.1; no longer S42.1
- net R1: now also D14.1 (K); no longer D26.1 (K), D27.1 (K)
- net R2: now also D26.1 (K), D77.1 (K); no longer D40.1 (K), D41.1 (K)
- net R3: now also D27.1 (K), D40.1 (K); no longer D54.1 (K), D55.1 (K)
- net R4: now also D41.1 (K), D54.1 (K); no longer D67.1 (K)
- net R5: now also D55.1 (K), D67.1 (K); no longer D14.1 (K), D77.1 (K)
Other:
- moved on the sheet: D14, D26, D27, D28, D40, D41, D42, D54, D55, D67, D77, S14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

Commit message: Add firmware
Parts:
- S27: value Add -> Equals
Other:
- moved on the sheet: D1, D10, D11, D12, D13, D14, D15, D16, D17, D18, D19, D2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
