File: PCB/PicoKeyboard/key_matrix.kicad_sch (KiCad schematic)
At the start: 154 parts

Commit message: Update PCB
Parts:
- S15: value Backtick -> Tilde
- S40: value [ -> LBrace
- S41: value ] -> RBrace
- S42: value Pipe -> BSlash
- S56: value L.Shift -> LShift
- S67: value R.Shift -> RShift
Changed lines of the file:
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@@
 			)
 		)
-		(property "Value" "R.Shift"
+		(property "Value" "RShift"
 			(at 214.63 205.74 0)
 			(effects
@@
 			)
 		)
-		(property "Value" "Backtick"
+		(property "Value" "Tilde"
 			(at 100.33 104.14 0)
 			(effects
@@
 			)
 		)
-		(property "Value" "]"
+		(property "Value" "RBrace"
 			(at 252.73 180.34 0)
 			(effects
@@
 			)
 		)
-		(property "Value" "L.Shift"
+		(property "Value" "LShift"
 			(at 100.33 180.34 0)
 			(effects
@@
 			)
 		)
-		(property "Value" "["
+		(property "Value" "LBrace"
 			(at 240.03 154.94 0)
 			(effects
@@
 			)
 		)
-		(property "Value" "Pipe"
+		(property "Value" "BSlash"
 			(at 240.03 205.74 0)
 			(effects
